File: Pmod_encoder/Pmod_encoder.kicad_pcb (KiCad board)
At the start: 2 copper layers, 38.6 x 19.8 mm, 11 parts, among them SW1 SW_SPDT, SW2 RotaryEncoder_Switch

Commit message: 605
Parts:
- moved R5 0.38 mm to (116.5, 85.5)
Routing:
- net Net-(R4-Pad2): track 28.3 -> 33.4 mm
- net Net-(R3-Pad2): track 44.7 -> 49.3 mm
- net Net-(R2-Pad2): track 30.9 -> 30.0 mm
- net GND: vias 1 -> 3
Other:
- board size 38.6 x 19.8 mm -> 39.1 x 19.8 mm
- board text added: "ver 0.2"
