File: Pmod_PLED/Pmod_PLED.kicad_pcb (KiCad board)
At the start: 2 copper layers, 75.8 x 20 mm, 7 parts, among them IC1 TBD62064APG, IC2 LM2940T-5.0, J1 Barrel_Jack_Switch, J2 Conn_01x06_Pin, J3 Conn_01x03_Pin

Commit message: 30
Parts:
- added Reserve: TestPoint, TestPoint:TestPoint_Pad_D2.0mm, F.Cu at (112.3, 89.7)
- D1: value EP204K-150G1R1B1-CA -> [EP204K-150G1R1B1-CA]
- J2: footprint Connector_PinHeader_2.54mm:PinHeader_1x06_P2.54mm_Vertical -> Library:Pmod6
- moved D3 22.5 mm to (138.8, 94.2)
- moved J2 9.40 mm to (83.8, 79.9)
- moved IC2 6.73 mm to (160.9, 83.9), turned to -90 degrees
- moved J3 2.29 mm to (134.1, 78.4)
- moved IC1 2.27 mm to (104.6, 82.3)
- moved D1 1.78 mm to (128.3, 86.4)
- moved J1 1.23 mm to (148.9, 91.6)
Connections:
- D1 pad 2: unconnected-(D1-RK-Pad2) -> Net-(IC1-O2)
- D1 pad 5: Net-(D1-A) -> unconnected-(D1-RK-Pad5)
- D1 pad 6: Net-(D1-A) -> /Anode
- D3 pad 2: Net-(D1-A) -> /Anode
- IC1 pad 14: GND -> Net-(IC1-I4)
- IC1 pad 16: unconnected-(IC1-O4-Pad16) -> Net-(IC1-O4)
- IC1 pad 7: unconnected-(IC1-O2-Pad7) -> Net-(IC1-O2)
- J2 pad 4: unconnected-(J2-Pin_4-Pad4) -> Net-(IC1-I4)
- J3 pad 2: Net-(D1-A) -> /Anode
Routing:
- net VCC: track 0.00 -> 53.1 mm
- net Net-(D1-BK): track 0.00 -> 28.1 mm
- net /ExVcc: track 0.00 -> 23.0 mm
- net Net-(IC1-O2): track 0.00 -> 22.9 mm
- net Net-(IC2-IN): track 0.00 -> 21.0 mm
- net /Anode: track 0.00 -> 20.9 mm
- net Net-(IC1-I1): track 0.00 -> 19.3 mm
- net Net-(IC1-I4): track 0.00 -> 17.6 mm
- net Net-(IC1-I2): track 0.00 -> 11.0 mm
- net Net-(IC1-I3): track 0.00 -> 9.88 mm
- net Net-(D1-GK): track 0.00 -> 8.95 mm
- net Net-(IC1-O4): track 0.00 -> 4.08 mm
- net Net-(D1-RA): track 0.00 -> 3.87 mm
- added copper zone on B.Cu, net GND
- added copper zone on F.Cu, net GND
Other:
- board size 75.8 x 20 mm -> 74.4 x 20.3 mm
- board text added: "[EP204K- 150G1R1B1-CA]"

Commit message: 30
Routing:
- net Net-(D1-BK): track 28.1 -> 26.3 mm
Other:
- board size 74.4 x 20.3 mm -> 74.5 x 20.3 mm
- board text added: "Pmod_Color_LED Ver. 0.1"
Changed lines of the file:
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@@
     )
   )
-  (gr_rect (start 88.458 76.073) (end 162.875 96.393)
+  (gr_arc (start 146.050643 76.079129) (mid 145.550643 76.579129) (end 145.050643 76.079129)
+    (stroke (width 0.1) (type default)) (layer "Edge.Cuts"))
+  (gr_line (start 145.058865 96.381837) (end 88.458 96.393)
+    (stroke (width 0.1) (type default)) (layer "Edge.Cuts"))
+  (gr_arc (start 145.052687 96.386938) (mid 145.552687 95.886938) (end 146.052687 96.386938)
+    (stroke (width 0.1) (type default)) (layer "Edge.Cuts"))
+  (gr_line (start 146.047999 90.287) (end 146.047999 80.1)
+    (stroke (width 0.1) (type default)) (layer "Edge.Cuts"))
+  (gr_line (start 146.05 76.074368) (end 162.896428 76.071986)
+    (stroke (width 0.1) (type default)) (layer "Edge.Cuts"))
+  (gr_circle (center 145.550648 94.4) (end 146.050648 94.4)
     (stroke (width 0.1) (type default)) (fill none) (layer "Edge.Cuts"))
+  (gr_circle (center 145.550648 92.4) (end 146.050648 92.4)
+    (stroke (width 0.1) (type default)) (fill none) (layer "Edge.Cuts"))
+  (gr_arc (start 146.047999 90.287) (mid 145.547999 90.787) (end 145.047999 90.287)
+    (stroke (width 0.1) (type default)) (layer "Edge.Cuts"))
+  (gr_line (start 145.047999 90.287) (end 145.047999 80.1)
+    (stroke (width 0.1) (type default)) (layer "Edge.Cuts"))
+  (gr_line (start 162.9 76.073772) (end 162.902308 96.39147)
+    (stroke (width 0.1) (type default)) (layer "Edge.Cuts"))
+  (gr_line (start 88.458 76.073) (end 145.049328 76.079429)
+    (stroke (width 0.1) (type default)) (layer "Edge.Cuts"))
+  (gr_line (start 88.449735 76.067821) (end 88.455542 96.392061)
+    (stroke (width 0.1) (type default)) (layer "Edge.Cuts"))
+  (gr_line (start 162.902308 96.39147) (end 146.047999 96.387396)
+    (stroke (width 0.1) (type default)) (layer "Edge.Cuts"))
+  (gr_arc (start 145.047999 80.1) (mid 145.547999 79.6) (end 146.047999 80.1)
+    (stroke (width 0.1) (type default)) (layer "Edge.Cuts"))
   (gr_text "[EP204K-\n 150G1R1B1-CA]" (at 136.779 93.853) (layer "B.SilkS")
     (effects (font (size 1.2 1.2) (thickness 0.15)) (justify left bottom mirror))
+  )
+  (gr_text "Pmod_Color_LED Ver. 0.1" (at 96.52 95.758) (layer "F.SilkS")
+    (effects (font (size 1.5 1.5) (thickness 0.3) bold) (justify left bottom))
   )
   (segment (start 110.998 78.486) (end 110.998 79.502) (width 0.5) (layer "F.Cu") (net 1))
@@
   (segment (start 102.997 83.185) (end 113.665 83.185) (width 0.5) (layer "F.Cu") (net 2))
   (segment (start 113.665 83.185) (end 116.888006 86.408006) (width 0.5) (layer "F.Cu") (net 2))
-  (segment (start 100.076 92.202) (end 118.418012 92.202) (width 0.5) (layer "F.Cu") (net 3))
   (segment (start 95.758 86.106) (end 95.758 87.884) (width 0.5) (layer "F.Cu") (net 3))
   (segment (start 95.758 87.884) (end 100.076 92.202) (width 0.5) (layer "F.Cu") (net 3))
-  (segment (start 118.418012 92.202) (end 119.712006 90.908006) (width 0.5) (layer "F.Cu") (net 3))
+  (segment (start 116.640012 92.202) (end 117.934006 90.908006) (width 0.5) (layer "F.Cu") (net 3))
+  (segment (start 100.076 92.202) (end 116.640012 92.202) (width 0.5) (layer "F.Cu") (net 3))
   (segment (start 137.311 92.231012) (end 138.634006 90.908006) (width 1) (layer "F.Cu") (net 4))
   (segment (start 137.311 94.234) (end 137.311 92.231012) (width 1) (layer "F.Cu") (net 4))
@@
     (polygon
       (pts
-        (xy 162.433 76.327)
-        (xy 162.433 96.139)
-        (xy 162.306 96.266)
-        (xy 88.646 96.266)
-        (xy 88.646 76.327)
+        (xy 162.733 76.727)
+        (xy 162.433 95.7)
+        (xy 162.106 95.666)
+        (xy 88.6 95.7)
+        (xy 88.6 76.7)
       )
     )
@@
     (polygon
       (pts
-        (xy 162.433 76.327)
-        (xy 162.433 96.139)
-        (xy 162.306 96.266)
-        (xy 88.646 96.266)
-        (xy 88.646 76.327)
-      )
-    )
+        (xy 162.633 76.727)
+        (xy 162.433 95.7)
+        (xy 162.406 95.666)
+        (xy 88.6 95.7)
+        (xy 88.6 76.7)
+      )
+    )

Commit message: 31
Connections:
- D1 pad 5: unconnected-(D1-RK-Pad5) -> Net-(IC1-O2)
Routing:
- net Net-(IC1-O2): track 22.9 -> 39.4 mm
- net VCC: track 53.1 -> 52.4 mm
- net Net-(IC2-IN): track 21.0 -> 21.7 mm
Other:
- outline, holes or cut-outs redrawn
- board text added: "1"
- board text added: "2"
- board text added: "3"
- board text added: "4"
- board text added: "Ex Vcc"
- board text added: "GND"
- board text added: "Vcc"
- board text added: "[LM2940T -3.3]"
- board text added: "[TBD62064APG]"
- board text added: "i1"
- board text added: "i2"
- board text added: "i3"
- board text added: "i4"
- board text added: "in"
- board text added: "o1"
- board text added: "o2"
- board text added: "o3"
- board text added: "o4"
- board text added: "out"

Commit message: 601
Parts:
- added G***: LOGO, MyLibrary:logo_kamo_ss, F.Cu at (152.5, 80.4)
- moved IC2 5.06 mm to (159.9, 79.0), turned to 90 degrees
- moved J2 4.89 mm to (88.5, 78.6)
- moved J1 0.32 mm to (148.9, 91.9)
Routing:
- net /ExVcc: track 23.0 -> 22.0 mm
- net Net-(IC2-IN): track 21.7 -> 22.4 mm
- net GND: vias 0 -> 3

Commit message: 601b
Parts:
- D1: value [EP204K-150G1R1B1-CA] -> EP204K-150G1R1B1-CA
- moved IC1 3.30 mm to (104.6, 85.6)
- moved TP1 2.41 mm to (112.3, 92.1)
- renumbered Reserve to TP1
Connections:
- D1 pad 5: Net-(IC1-O2) -> unconnected-(D1-RK-Pad5)
Routing:
- net Net-(IC1-O2): track 39.4 -> 21.8 mm
- net VCC: track 52.4 -> 62.2 mm
- net Net-(IC1-I1): track 19.3 -> 18.0 mm
- net Net-(IC1-O4): track 4.08 -> 3.19 mm
- net Net-(IC1-I4): track 17.6 -> 18.2 mm
- net Net-(D1-BK): track 26.6 -> 27.2 mm
- net Net-(IC1-I2): track 11.0 -> 10.4 mm
- net GND: vias 3 -> 0
- removed copper zone on B.Cu, net GND

Commit message: 601c
Parts:
- moved G*** 0.13 mm to (152.5, 80.5)
- renumbered TP1 to Reserve
Other:
- board text added: "ExVcc"
- board text removed: "Ex Vcc"
Changed lines of the file:
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@@
   )
   (footprint "MyLibrary:logo_kamo_ss" (layer "F.Cu")
-    (at 152.527 80.391)
+    (at 152.527 80.518)
     (attr board_only exclude_from_pos_files exclude_from_bom)
     (fp_text reference "G***" (at 0 0) (layer "F.SilkS") hide
@@
     (property "ki_keywords" "test point tp")
     (attr exclude_from_pos_files)
-    (fp_text reference "TP1" (at -4.445 -0.127) (layer "F.SilkS")
+    (fp_text reference "Reserve" (at -4.064 0.889) (layer "F.SilkS")
         (effects (font (size 1 1) (thickness 0.15)))
     )
     (fp_text value "TestPoint" (at -4.572 1.524) (layer "F.Fab")
-        (effects (font (size 1 1) (thickness 0.15)))
-    )
-    (fp_text user "${REFERENCE}" (at 0 -2) (layer "F.Fab")
         (effects (font (size 1 1) (thickness 0.15)))
     )
@@
     (property "ki_description" "Gate Drivers DMOS Transistor Array 4-CH 50V/1.5A")
     (attr through_hole)
-    (fp_text reference "IC1" (at 5.842 4.191 -180) (layer "F.SilkS")
+    (fp_text reference "IC1" (at 5.588 -0.254 -180) (layer "F.SilkS")
         (effects (font (size 1.27 1.27) (thickness 0.254)))
     )
@@
         (effects (font (size 1 1) (thickness 0.1)) (justify left bottom))
     )
-    (fp_text user "B" (at -13.780006 6.047994 unlocked) (layer "F.SilkS")
+    (fp_text user "B" (at -9.716006 7.063994 unlocked) (layer "F.SilkS")
         (effects (font (size 1 1) (thickness 0.1)) (justify left bottom))
     )
@@
   (gr_arc (start 145.047999 80.1) (mid 145.547999 79.6) (end 146.047999 80.1)
     (stroke (width 0.1) (type default)) (layer "Edge.Cuts"))
-  (gr_text "in" (at 157.734 79.121) (layer "B.SilkS")
+  (gr_text "in" (at 159.004 79.121) (layer "B.SilkS")
     (effects (font (size 1 1) (thickness 0.15)) (justify left bottom mirror))
   )
-  (gr_text "o1" (at 112.014 80.899) (layer "B.SilkS")
-    (effects (font (size 1 1) (thickness 0.125)) (justify left bottom mirror))
-  )
-  (gr_text "out" (at 157.734 84.836) (layer "B.SilkS")
+  (gr_text "out" (at 159.258 84.836) (layer "B.SilkS")
     (effects (font (size 1 1) (thickness 0.15)) (justify left bottom mirror))
-  )
-  (gr_text "i4" (at 109.22 84.963) (layer "B.SilkS")
-    (effects (font (size 1 1) (thickness 0.125)) (justify left bottom mirror))
-  )
-  (gr_text "o4" (at 114.427 84.963) (layer "B.SilkS")
-    (effects (font (size 1 1) (thickness 0.125)) (justify left bottom mirror))
   )
   (gr_text "[LM2940T\n   -3.3]" (at 157.734 82.677) (layer "B.SilkS")
@@
     (effects (font (size 1 1) (thickness 0.15)) (justify left bottom mirror))
   )
+  (gr_text "GND" (at 97.028 91.44) (layer "B.SilkS")
+    (effects (font (size 1 1) (thickness 0.15)) (justify left bottom mirror))
+  )
   (gr_text "2" (at 90.551 83.058) (layer "B.SilkS")
     (effects (font (size 1 1) (thickness 0.15)) (justify left bottom mirror))
   )
-  (gr_text "o3" (at 96.774 84.963) (layer "B.SilkS")
-    (effects (font (size 1 1) (thickness 0.125)) (justify left bottom mirror))
-  )
-  (gr_text "i1" (at 109.093 80.899) (layer "B.SilkS")
-    (effects (font (size 1 1) (thickness 0.125)) (justify left bottom mirror))
-  )
   (gr_text "3" (at 90.551 85.598) (layer "B.SilkS")
     (effects (font (size 1 1) (thickness 0.15)) (justify left bottom mirror))
   )
-  (gr_text "o2" (at 99.314 80.645) (layer "B.SilkS")
-    (effects (font (size 1 1) (thickness 0.125)) (justify left bottom mirror))
-  )
-  (gr_text "i3" (at 101.6 84.963) (layer "B.SilkS")
-    (effects (font (size 1 1) (thickness 0.125)) (justify left bottom mirror))
-  )
   (gr_text "1" (at 90.551 80.518) (layer "B.SilkS")
     (effects (font (size 1 1) (thickness 0.15)) (justify left bottom mirror))
@@
     (effects (font (size 1.2 1.2) (thickness 0.15)) (justify left bottom mirror))
   )
-  (gr_text "i2" (at 101.6 80.645) (layer "B.SilkS")
-    (effects (font (size 1 1) (thickness 0.125)) (justify left bottom mirror))
+  (gr_text "o1" (at 110.236 80.772) (layer "F.SilkS")
+    (effects (font (size 1 1) (thickness 0.125)) (justify left bottom))
+  )
+  (gr_text "i4" (at 107.95 91.694) (layer "F.SilkS")
+    (effects (font (size 1 1) (thickness 0.125)) (justify left bottom))
+  )
+  (gr_text "o4" (at 113.538 91.44) (layer "F.SilkS")
+    (effects (font (size 1 1) (thickness 0.125)) (justify left bottom))
   )
   (gr_text "Pmod_Color_LED Ver. 0.1" (at 96.52 95.758) (layer "F.SilkS")
     (effects (font (size 1.5 1.5) (thickness 0.3) bold) (justify left bottom))
   )
-  (gr_text "GND" (at 94.107 90.551) (layer "F.SilkS")
+  (gr_text "ExVcc" (at 140.462 79.121) (layer "F.SilkS")
+    (effects (font (size 1.4 1.4) (thickness 0.175)) (justify left bottom))
+  )
+  (gr_text "o3" (at 94.996 91.694) (layer "F.SilkS")
+    (effects (font (size 1 1) (thickness 0.125)) (justify left bottom))
+  )
+  (gr_text "i1" (at 107.696 80.772) (layer "F.SilkS")
+    (effects (font (size 1 1) (thickness 0.125)) (justify left bottom))
+  )
+  (gr_text "Vcc" (at 93.98 93.218) (layer "F.SilkS")
     (effects (font (size 1 1) (thickness 0.15)) (justify left bottom))
   )
-  (gr_text "Ex Vcc" (at 140.462 79.121) (layer "F.SilkS")
-    (effects (font (size 1.4 1.4) (thickness 0.175)) (justify left bottom))
-  )
-  (gr_text "Vcc" (at 94.234 93.091) (layer "F.SilkS")
+  (gr_text "o2" (at 97.028 80.645) (layer "F.SilkS")
+    (effects (font (size 1 1) (thickness 0.125)) (justify left bottom))
+  )
+  (gr_text "[TBD62064APG]" (at 99.441 86.36) (layer "F.SilkS")
     (effects (font (size 1 1) (thickness 0.15)) (justify left bottom))
   )
-  (gr_text "[TBD62064APG]" (at 99.441 82.804) (layer "F.SilkS")
-    (effects (font (size 1 1) (thickness 0.15)) (justify left bottom))
+  (gr_text "i3" (at 100.076 91.694) (layer "F.SilkS")
+    (effects (font (size 1 1) (thickness 0.125)) (justify left bottom))
   )
   (gr_text "Vcc" (at 128.778 78.994) (layer "F.SilkS")
     (effects (font (size 1.4 1.4) (thickness 0.175)) (justify left bottom))
   )
+  (gr_text "i2" (at 100.076 80.645) (layer "F.SilkS")
+    (effects (font (size 1 1) (thickness 0.125)) (justify left bottom))
+  )
   (segment (start 116.211994 81.908006) (end 117.934006 81.908006) (width 0.5) (layer "F.Cu") (net 1))

Commit message: 601d
Other:
- outline, holes or cut-outs redrawn
Changed lines of the file:
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@@
     (fp_circle (center 0 0) (end 1.5 0)
       (stroke (width 0.05) (type solid)) (fill none) (layer "F.CrtYd"))
-    (pad "" np_thru_hole circle (at 0 0) (size 1.8 1.8) (drill 1) (layers "F&B.Cu" "*.Mask")
+    (pad "" np_thru_hole circle (at 0 0) (size 1.6 1.6) (drill 1) (layers "F&B.Cu" "*.Mask")
       (pinfunction "1") (pintype "passive"))
   )
@@
     (fp_line (start 2.7432 2.8448) (end 2.7432 -1.8288)
       (stroke (width 0.1524) (type solid)) (layer "F.Fab"))
-    (pad "" np_thru_hole rect (at -5.08 1.016 90) (size 1.905 1.905) (drill 1.27) (layers "F&B.Cu" "*.Mask")
+    (pad "" np_thru_hole rect (at -5.08 1.016 90) (size 1.905 1.905) (drill 1) (layers "F&B.Cu" "*.Mask")
       (pinfunction "IN") (pintype "passive"))
-    (pad "" np_thru_hole circle (at -2.54 1.016 90) (size 1.905 1.905) (drill 1.27) (layers "F&B.Cu" "*.Mask")
+    (pad "" np_thru_hole circle (at -2.54 1.016 90) (size 1.905 1.905) (drill 1) (layers "F&B.Cu" "*.Mask")
       (pinfunction "GND") (pintype "passive"))
-    (pad "" np_thru_hole circle (at 0 1.016 90) (size 1.905 1.905) (drill 1.27) (layers "F&B.Cu" "*.Mask")
+    (pad "" np_thru_hole circle (at 0 1.016 90) (size 1.905 1.905) (drill 1) (layers "F&B.Cu" "*.Mask")
       (pinfunction "OUT") (pintype "passive"))
     (model "C:\\Users\\n11ak\\Documents\\kicad\\7.0\\SamacSys_Parts.3dshapes\\LM2940T-5.0.stp"
@@
     (pad "" np_thru_hole rect (at -3.81 -8.89 270) (size 1.2 1.2) (drill 0.8) (layers "F&B.Cu" "*.Mask")
       (pinfunction "COMMON_1") (pintype "passive+no_connect"))
-    (pad "" np_thru_hole circle (at -3.81 -6.35 270) (size 1.2 1.2) (drill 0.8) (layers "F&B.Cu" "*.Mask")
+    (pad "" np_thru_hole oval (at -3.81 -6.35 270) (size 1.6 1.2) (drill 1) (layers "F&B.Cu" "*.Mask")
       (pinfunction "O1") (pintype "passive"))
-    (pad "" np_thru_hole circle (at -3.81 -3.81 270) (size 1.2 1.2) (drill 0.8) (layers "F&B.Cu" "*.Mask")
+    (pad "" np_thru_hole oval (at -3.81 -3.81 270) (size 1.6 1.2) (drill 1) (layers "F&B.Cu" "*.Mask")
       (pinfunction "I1") (pintype "passive"))
-    (pad "" np_thru_hole circle (at -3.81 -1.27 270) (size 1.2 1.2) (drill 0.8) (layers "F&B.Cu" "*.Mask")
+    (pad "" np_thru_hole oval (at -3.81 -1.27 270) (size 1.5 1.3) (drill 1) (layers "F&B.Cu" "*.Mask")
       (pinfunction "GND_1") (pintype "passive"))
-    (pad "" np_thru_hole circle (at -3.81 1.27 270) (size 1.2 1.2) (drill 0.8) (layers "F&B.Cu" "*.Mask")
+    (pad "" np_thru_hole oval (at -3.81 1.27 270) (size 1.5 1.3) (drill 1) (layers "F&B.Cu" "*.Mask")
       (pinfunction "GND_2") (pintype "passive"))
-    (pad "" np_thru_hole circle (at -3.81 3.81 270) (size 1.2 1.2) (drill 0.8) (layers "F&B.Cu" "*.Mask")
+    (pad "" np_thru_hole oval (at -3.81 3.81 270) (size 1.5 1.3) (drill 1) (layers "F&B.Cu" "*.Mask")
       (pinfunction "I2") (pintype "passive"))
-    (pad "" np_thru_hole circle (at -3.81 6.35 270) (size 1.2 1.2) (drill 0.8) (layers "F&B.Cu" "*.Mask")
+    (pad "" np_thru_hole oval (at -3.81 6.35 270) (size 1.5 1.4) (drill 1) (layers "F&B.Cu" "*.Mask")
       (pinfunction "O2") (pintype "passive"))
-    (pad "" np_thru_hole circle (at -3.81 8.89 270) (size 1.2 1.2) (drill 0.8) (layers "F&B.Cu" "*.Mask")
+    (pad "" np_thru_hole oval (at -3.81 8.89 270) (size 1.5 1.4) (drill 1) (layers "F&B.Cu" "*.Mask")
       (pinfunction "COMMON_2") (pintype "passive+no_connect"))
-    (pad "" np_thru_hole circle (at 3.81 -8.89 270) (size 1.2 1.2) (drill 0.8) (layers "F&B.Cu" "*.Mask")
+    (pad "" np_thru_hole oval (at 3.81 -8.89 270) (size 1.5 1.3) (drill 1) (layers "F&B.Cu" "*.Mask")
       (pinfunction "O4") (pintype "passive"))
     (pad "" np_thru_hole circle (at 3.81 -6.35 270) (size 1 1) (drill 1) (layers "F&B.Cu" "*.Mask")
       (pinfunction "NC_2") (pintype "passive+no_connect"))
-    (pad "" np_thru_hole circle (at 3.81 -3.81 270) (size 1.2 1.2) (drill 0.8) (layers "F&B.Cu" "*.Mask")
+    (pad "" np_thru_hole oval (at 3.81 -3.81 270) (size 1.5 1.3) (drill 1) (layers "F&B.Cu" "*.Mask")
       (pinfunction "I4") (pintype "passive"))
-    (pad "" np_thru_hole circle (at 3.81 -1.27 270) (size 1.2 1.2) (drill 0.8) (layers "F&B.Cu" "*.Mask")
+    (pad "" np_thru_hole oval (at 3.81 -1.27 270) (size 1.5 1.3) (drill 1) (layers "F&B.Cu" "*.Mask")
       (pinfunction "GND_4") (pintype "passive"))
-    (pad "" np_thru_hole circle (at 3.81 1.27 270) (size 1.2 1.2) (drill 0.8) (layers "F&B.Cu" "*.Mask")
+    (pad "" np_thru_hole oval (at 3.81 1.27 270) (size 1.5 1.3) (drill 1) (layers "F&B.Cu" "*.Mask")
       (pinfunction "GND_3") (pintype "passive"))
-    (pad "" np_thru_hole circle (at 3.81 3.81 270) (size 1.2 1.2) (drill 0.8) (layers "F&B.Cu" "*.Mask")
+    (pad "" np_thru_hole oval (at 3.81 3.81 270) (size 1.5 1.3) (drill 1) (layers "F&B.Cu" "*.Mask")
       (pinfunction "I3") (pintype "passive"))
     (pad "" np_thru_hole circle (at 3.81 6.35 270) (size 1 1) (drill 1) (layers "F&B.Cu" "*.Mask")
       (pinfunction "NC_1") (pintype "passive+no_connect"))
-    (pad "" np_thru_hole circle (at 3.81 8.89 270) (size 1.2 1.2) (drill 0.8) (layers "F&B.Cu" "*.Mask")
+    (pad "" np_thru_hole oval (at 3.81 8.89 270) (size 1.5 1.3) (drill 1) (layers "F&B.Cu" "*.Mask")
       (pinfunction "O3") (pintype "passive"))
     (model "C:\\Users\\n11ak\\Documents\\kicad\\7.0\\SamacSys_Parts.3dshapes\\TBD62064APG.stp"
@@
   (gr_rect (start 129.667 83.82) (end 137.541 88.9)
     (stroke (width 0.2) (type solid)) (fill solid) (layer "F.Cu"))
-  (gr_line (start 153.924 91.059) (end 152.527 88.138)
-    (stroke (width 1) (type default)) (layer "F.Cu"))
   (gr_rect (start 119.253 83.82) (end 127.127 88.9)
     (stroke (width 0.2) (type solid)) (fill solid) (layer "F.Cu"))
-  (gr_arc (start 146.05 76.066291) (mid 145.550643 76.565648) (end 145.051286 76.066291)
-    (stroke (width 0.1) (type default)) (layer "Edge.Cuts"))
-  (gr_line (start 145.042536 96.381607) (end 88.439228 96.381607)
-    (stroke (width 0.1) (type default)) (layer "Edge.Cuts"))
-  (gr_arc (start 145.042536 96.381607) (mid 145.542536 95.881607) (end 146.042536 96.381607)
-    (stroke (width 0.1) (type default)) (layer "Edge.Cuts"))
-  (gr_line (start 146.047999 90.287) (end 146.047999 80.1)
-    (stroke (width 0.1) (type default)) (layer "Edge.Cuts"))
-  (gr_line (start 146.05 76.066291) (end 162.896428 76.063909)
-    (stroke (width 0.1) (type default)) (layer "Edge.Cuts"))
-  (gr_circle (center 145.550648 94.4) (end 146.050648 94.4)
+  (gr_arc (start 145.660357 76.066291) (mid 145.161 76.565648) (end 144.661643 76.066291)
+    (stroke (width 0.1) (type default)) (layer "Edge.Cuts"))
+  (gr_line (start 144.915 96.381607) (end 88.439228 96.381607)
+    (stroke (width 0.1) (type default)) (layer "Edge.Cuts"))
+  (gr_arc (start 144.915 96.381607) (mid 145.415 95.881607) (end 145.915 96.381607)
+    (stroke (width 0.1) (type default)) (layer "Edge.Cuts"))
+  (gr_line (start 146.292002 90.287) (end 146.298001 80.512001)
+    (stroke (width 0.1) (type default)) (layer "Edge.Cuts"))
+  (gr_line (start 145.660357 76.066291) (end 162.896428 76.063909)
+    (stroke (width 0.1) (type default)) (layer "Edge.Cuts"))
+  (gr_circle (center 145.415 94.488) (end 145.915 94.488)
     (stroke (width 0.1) (type default)) (fill none) (layer "Edge.Cuts"))
-  (gr_circle (center 145.550648 92.4) (end 146.050648 92.4)
+  (gr_circle (center 145.415 92.464) (end 145.915 92.464)
     (stroke (width 0.1) (type default)) (fill none) (layer "Edge.Cuts"))
-  (gr_arc (start 146.047999 90.287) (mid 145.547999 90.787) (end 145.047999 90.287)
-    (stroke (width 0.1) (type default)) (layer "Edge.Cuts"))
-  (gr_line (start 145.047999 90.287) (end 145.047999 80.1)
+  (gr_arc (start 146.292002 90.287) (mid 145.282001 91.297001) (end 144.272 90.287)
+    (stroke (width 0.1) (type default)) (layer "Edge.Cuts"))
+  (gr_line (start 144.272 90.287) (end 144.277999 80.512001)
     (stroke (width 0.1) (type default)) (layer "Edge.Cuts"))
   (gr_line (start 162.896428 76.063909) (end 162.898736 96.381607)
     (stroke (width 0.1) (type default)) (layer "Edge.Cuts"))
-  (gr_line (start 88.4428 76.066291) (end 145.051286 76.066291)
+  (gr_line (start 88.4428 76.066291) (end 144.661643 76.066291)
+    (stroke (width 0.1) (type default)) (layer "Edge.Cuts"))
+  (gr_arc (start 144.277999 80.512001) (mid 145.288 79.502) (end 146.298001 80.512001)
     (stroke (width 0.1) (type default)) (layer "Edge.Cuts"))
   (gr_line (start 88.439228 76.2) (end 88.439228 96.381607)
@@
   (gr_line (start 88.439228 76.2) (end 88.439228 76.066291)
     (stroke (width 0.1) (type default)) (layer "Edge.Cuts"))
-  (gr_line (start 162.898736 96.381607) (end 146.042536 96.381607)
-    (stroke (width 0.1) (type default)) (layer "Edge.Cuts"))
-  (gr_arc (start 145.047999 80.1) (mid 145.547999 79.6) (end 146.047999 80.1)
+  (gr_line (start 162.898736 96.381607) (end 145.915 96.381607)
     (stroke (width 0.1) (type default)) (layer "Edge.Cuts"))
   (gr_text "in" (at 159.004 79.121) (layer "B.SilkS")
