File: Pmod_PLED/Pmod_PLED.kicad_pcb (KiCad board)
At the start: 2 copper layers, 74.5 x 20.3 mm, 9 parts, among them IC1 TBD62064APG, IC2 LM2940T-5.0, J1 Barrel_Jack_Switch, J2 Conn_01x06_Pin, J3 Conn_01x03_Pin

Commit message: 613
Parts:
- moved G*** 0.52 mm to (152.4, 81.0)
- moved D3 0.51 mm to (138.8, 93.7)
- moved IC2 0.34 mm to (160.1, 79.2)
- moved J1 0.25 mm to (149.2, 91.9)
Connections:
- IC1 pad : (no net) -> Net-(D1-BK)
- IC2 pad : (no net) -> /ExVcc
- J1 pad : (no net) -> Net-(IC2-IN)
- J2 pad : (no net) -> VCC
- J3 pad : (no net) -> /ExVcc
- Reserve pad : (no net) -> Net-(IC1-O4)
Routing:
- net Net-(IC2-IN): track 22.4 -> 24.7 mm
- net Net-(IC1-I2): track 10.4 -> 11.6 mm
- net Net-(D1-RA): track 3.87 -> 3.37 mm
Other:
- board text added: "Pmod_Color_LED Ver. 0.2"
- board text removed: "Pmod_Color_LED Ver. 0.1"
