File: Pmod_PLED/Pmod_PLED.kicad_pcb (KiCad board)
At the start: 2 copper layers, 74.5 x 20.3 mm, 9 parts, among them IC1 TBD62064APG, IC2 LM2940T-5.0, J1 Barrel_Jack_Switch, J2 Conn_01x06_Pin, J3 Conn_01x03_Pin

Commit message: 617
Parts:
- removed IC2: LM2940T-5.0, SamacSys_Parts:TO254P470X1016X2222-3P
- added U1: AMS1117-3.3, Package_TO_SOT_SMD:SOT-223-3_TabPin2, F.Cu at (158.8, 81.8)
- G***: moved to B.Cu
- moved G*** 47.4 mm to (105.2, 85.1), turned to 180 degrees
- renumbered Reserve to TP1
Connections:
- net Net-(IC1-O4) renamed o4
- net VCC renamed vcc
Routing:
- net i1: track 0.00 -> 18.4 mm
- net Net-(IC1-I1): track 18.4 -> 0.00 mm
- net i4: track 0.00 -> 18.2 mm
- net Net-(IC1-I4): track 18.2 -> 0.00 mm
- net i2: track 0.00 -> 11.6 mm
- net Net-(IC1-I2): track 11.6 -> 0.00 mm
- net i3: track 0.00 -> 10.1 mm
- net Net-(IC1-I3): track 10.1 -> 0.00 mm
- net /ExVcc: track 22.0 -> 19.7 mm
- net Net-(U1-VI): track 24.7 -> 23.5 mm
- net Net-(IC1-O2): track 21.5 -> 22.4 mm
Other:
- board text added: "[AZ1117 CH-3.3]"
- board text removed: "[LM2940T -3.3]"

Commit message: 618
Parts:
- removed TP1: TestPoint, TestPoint:TestPoint_Pad_D2.0mm
- added C1: 0.1u, Capacitor_SMD:C_0603_1608Metric_Pad1.08x0.95mm_HandSolder, F.Cu at (160.2, 85.2)
- added C2: 0.1u, Capacitor_SMD:C_0603_1608Metric_Pad1.08x0.95mm_HandSolder, F.Cu at (148.2, 79.2)
- moved U1 4.36 mm to (154.5, 80.9), turned to 180 degrees
- moved J1 0.31 mm to (149.2, 91.6)
- moved IC1 0.25 mm to (104.6, 85.3)
Routing:
- net Net-(IC1-O4): track 22.4 -> 6.20 mm
- net Net-(U1-VI): track 23.5 -> 32.8 mm
- net /ExVcc: track 19.7 -> 13.2 mm
- net o4: track 3.19 -> 0.00 mm
- net i4: track 18.2 -> 19.4 mm
- net i2: track 11.6 -> 10.4 mm
- net i3: track 10.1 -> 11.0 mm
- net i1: track 18.4 -> 17.8 mm
