File: Pmod_PLED/Pmod_PLED.kicad_sch (KiCad schematic)
At the start: 1 part

Commit message: 29
Parts:
- added IC1: TBD62064APG, DIP762W60P254L1975H445Q16N, symbol SamacSys_Parts:TBD62064APG
- added IC2: LM2940T-5.0, TO254P470X1016X2222-3P, symbol SamacSys_Parts:LM2940T-5.0
- added J1: Barrel_Jack_Switch, Connector_BarrelJack:BarrelJack_Horizontal, symbol Connector:Barrel_Jack_Switch
Changed lines of the file:
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@@
+    )
+  )
+  (symbol (lib_id "SamacSys_Parts:TBD62064APG") (at 110.49 109.22 90) (unit 1)
+    (in_bom yes) (on_board yes) (dnp no) (fields_autoplaced)
+    (property "Reference" "IC1" (at 132.715 90.805 90)
+      (effects (font (size 1.27 1.27)) (justify right))
+    )
+    (property "Value" "TBD62064APG" (at 132.715 93.345 90)
+      (effects (font (size 1.27 1.27)) (justify right))
+    )
+    (property "Footprint" "DIP762W60P254L1975H445Q16N" (at 107.95 77.47 0)
+      (effects (font (size 1.27 1.27)) (justify left) hide)
+    )
+    (property "Datasheet" "https://toshiba.semicon-storage.com/info/docget.jsp?did=30810&prodName=TBD62064APG" (at 110.49 77.47 0)
+      (effects (font (size 1.27 1.27)) (justify left) hide)
+    )
+    (property "Description" "Gate Drivers DMOS Transistor Array 4-CH 50V/1.5A" (at 113.03 77.47 0)
+      (effects (font (size 1.27 1.27)) (justify left) hide)
+    )
+    (property "Height" "4.45" (at 115.57 77.47 0)
+      (effects (font (size 1.27 1.27)) (justify left) hide)
+    )
+    (property "RS Part Number" "" (at 118.11 77.47 0)
+      (effects (font (size 1.27 1.27)) (justify left) hide)
+    )
+    (property "RS Price/Stock" "" (at 120.65 77.47 0)
+      (effects (font (size 1.27 1.27)) (justify left) hide)
+    )
+    (property "Manufacturer_Name" "Toshiba" (at 123.19 77.47 0)
+      (effects (font (size 1.27 1.27)) (justify left) hide)
+    )
+    (property "Manufacturer_Part_Number" "TBD62064APG" (at 125.73 77.47 0)
+      (effects (font (size 1.27 1.27)) (justify left) hide)
+    )
+    (pin "1")
+    (pin "10")
+    (pin "11")
+    (pin "12")
+    (pin "13")
+    (pin "14")
+    (pin "15")
+    (pin "16")
+    (pin "2")
+    (pin "3")
+    (pin "4")
+    (pin "5")
+    (pin "6")
+    (pin "7")
+    (pin "8")
+    (pin "9")
+    (instances
+      (project "Pmod_PLED"
+        (path "/d5200c1e-908a-4e72-95f9-aca3b7bcc08a"
+          (reference "IC1") (unit 1)
+        )
+      )
+    )
+  )
+  (symbol (lib_id "SamacSys_Parts:LM2940T-5.0") (at 147.955 50.8 0) (unit 1)
+    (in_bom yes) (on_board yes) (dnp no) (fields_autoplaced)
+    (property "Reference" "IC2" (at 167.005 52.705 0)
+      (effects (font (size 1.27 1.27)) (justify left))
+    )
+    (property "Value" "LM2940T-5.0" (at 167.005 55.245 0)
+      (effects (font (size 1.27 1.27)) (justify left))
+    )
+    (property "Footprint" "TO254P470X1016X2222-3P" (at 167.005 48.26 0)
+      (effects (font (size 1.27 1.27)) (justify left) hide)
+    )
+    (property "Datasheet" "http://uk.rs-online.com/web/p/products/0411769" (at 167.005 50.8 0)
+      (effects (font (size 1.27 1.27)) (justify left) hide)
+    )
+    (property "Description" "IC, LDO VOLT REG, 5V, 1A" (at 167.005 53.34 0)
+      (effects (font (size 1.27 1.27)) (justify left) hide)
+    )
+    (property "Height" "" (at 167.005 55.88 0)
+      (effects (font (size 1.27 1.27)) (justify left) hide)
+    )
+    (property "RS Part Number" "0411769" (at 167.005 58.42 0)
+      (effects (font (size 1.27 1.27)) (justify left) hide)
+    )
+    (property "RS Price/Stock" "http://uk.rs-online.com/web/p/products/0411769" (at 167.005 60.96 0)
+      (effects (font (size 1.27 1.27)) (justify left) hide)
+    )
+    (property "Manufacturer_Name" "Texas Instruments" (at 167.005 63.5 0)
+      (effects (font (size 1.27 1.27)) (justify left) hide)
+    )
+    (property "Manufacturer_Part_Number" "LM2940T-5.0" (at 167.005 66.04 0)
+      (effects (font (size 1.27 1.27)) (justify left) hide)
+    )
+    (pin "1")
+    (pin "2")
+    (pin "3")
+    (instances
+      (project "Pmod_PLED"
+        (path "/d5200c1e-908a-4e72-95f9-aca3b7bcc08a"
+          (reference "IC2") (unit 1)
+        )
+      )
+    )
+  )
+  (symbol (lib_id "Connector:Barrel_Jack_Switch") (at 116.84 48.895 0) (unit 1)
+    (in_bom yes) (on_board yes) (dnp no) (fields_autoplaced)
+    (property "Reference" "J1" (at 116.84 40.64 0)
+      (effects (font (size 1.27 1.27)))
+    )
+    (property "Value" "Barrel_Jack_Switch" (at 116.84 43.18 0)
+      (effects (font (size 1.27 1.27)))
+    )
+    (property "Footprint" "Connector_BarrelJack:BarrelJack_Horizontal" (at 118.11 49.911 0)
+      (effects (font (size 1.27 1.27)) hide)
+    )
+    (property "Datasheet" "~" (at 118.11 49.911 0)
+      (effects (font (size 1.27 1.27)) hide)
+    )
+    (pin "1")
+    (pin "2")
+    (pin "3")
+    (instances
+      (project "Pmod_PLED"
+        (path "/d5200c1e-908a-4e72-95f9-aca3b7bcc08a"
+          (reference "J1") (unit 1)
+        )
+      )
     )
   )

Commit message: 29
Parts:
- added D3: SS2040FL, SamacSys_Parts:SODFL3618X108N, symbol SamacSys_Parts:SS2040FL
- added J2: Conn_01x06_Pin, Connector_PinHeader_2.54mm:PinHeader_1x06_P2.54mm_Vertical, symbol Connector:Conn_01x06_Pin
- added J3: Conn_01x03_Pin, Connector_PinHeader_2.54mm:PinHeader_1x03_P2.54mm_Vertical, symbol Connector:Conn_01x03_Pin
- D1: footprint (none) -> MyLibrary:EP204-150G1R1B1-CA
- IC1: footprint DIP762W60P254L1975H445Q16N -> SamacSys_Parts:DIP762W60P254L1975H445Q16N
- IC2: footprint TO254P470X1016X2222-3P -> SamacSys_Parts:TO254P470X1016X2222-3P
Connections:
- net at D1.1 (GK): now also IC1.2 (O1)
- net at D1.3 (BK): now also IC1.9 (O3)
- net at D1.4 (RA): now also D3.1 (K)
- net at D1.5 (RK): now also D1.6 (A), D3.2 (A), J3.2 (Pin_2)
- net at IC1.11 (I3): now also J2.3 (Pin_3)
- net GND: now reaches IC1.12 (GND_3)
- net GND: now also IC1.13 (GND_4), IC1.14 (I4), IC1.4 (GND_1), IC1.5 (GND_2), IC2.2 (GND), J1.2, J2.5 (Pin_5)
- net at IC1.3 (I1): now also J2.1 (Pin_1)
- net at IC1.6 (I2): now also J2.2 (Pin_2)
- net at IC2.1 (IN): now also J1.1
- net ExVcc: now reaches IC2.3 (OUT)
- net ExVcc: now also J3.3 (Pin_3)
- new net VCC: J2.6 (Pin_6), J3.1 (Pin_1)
- no-connect marks 0 -> 6
Other:
- moved on the sheet: IC1, IC2, J1

Commit message: 30
Parts:
- added TP1: TestPoint, TestPoint:TestPoint_Pad_D2.0mm, symbol Connector:TestPoint
- J2: footprint Connector_PinHeader_2.54mm:PinHeader_1x06_P2.54mm_Vertical -> Library:Pmod6
Connections:
- net GND: no longer IC1.14 (I4)
- net Anode: now reaches D1.6 (A), D3.2 (A), J3.2 (Pin_2)
- net Anode: no longer D1.5 (RK)
- net at J2.4 (Pin_4): now also IC1.14 (I4)
- net at D1.2 (RK): now also IC1.7 (O2)
- net at IC1.16 (O4): now also TP1.1
- no-connect marks 6 -> 4
Other:
- moved on the sheet: D1, D3, IC2, J1, J3

Commit message: 601b
Connections:
- net at J2.3 (Pin_3): now also IC1.14 (I4); no longer IC1.11 (I3)
- net at J2.4 (Pin_4): now also IC1.11 (I3); no longer IC1.14 (I4)
Changed lines of the file:
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@@
+    (stroke (width 0) (type default))
+  )
+  (wire (pts (xy 87.63 112.395) (xy 87.63 90.17))
     (stroke (width 0) (type default))
   )
@@
     (stroke (width 0) (type default))
   )
+  (wire (pts (xy 87.63 90.17) (xy 74.295 90.17))
+    (stroke (width 0) (type default))
+  )
   (wire (pts (xy 74.295 100.33) (xy 77.47 100.33))
     (stroke (width 0) (type default))
   )
   (wire (pts (xy 122.555 62.865) (xy 122.555 71.755))
+    (stroke (width 0) (type default))
+  )
+  (wire (pts (xy 86.36 87.63) (xy 74.295 87.63))
     (stroke (width 0) (type default))
   )
@@
     (stroke (width 0) (type default))
   )
-  (wire (pts (xy 87.63 87.63) (xy 87.63 112.395))
-    (stroke (width 0) (type default))
-  )
   (wire (pts (xy 122.555 113.665) (xy 122.555 107.315))
     (stroke (width 0) (type default))
@@
     (stroke (width 0) (type default))
   )
-  (wire (pts (xy 86.36 90.17) (xy 86.36 113.665))
+  (wire (pts (xy 86.36 87.63) (xy 86.36 113.665))
     (stroke (width 0) (type default))
   )
@@
   )
   (wire (pts (xy 120.015 71.755) (xy 118.745 71.755))
-    (stroke (width 0) (type default))
-  )
-  (wire (pts (xy 74.295 90.17) (xy 86.36 90.17))
     (stroke (width 0) (type default))
   )
@@
     (stroke (width 0) (type default))
   )
-  (wire (pts (xy 74.295 87.63) (xy 87.63 87.63))
-    (stroke (width 0) (type default))
-  )

Commit message: 617
Parts:
- removed IC2: LM2940T-5.0, SamacSys_Parts:TO254P470X1016X2222-3P, symbol SamacSys_Parts:LM2940T-5.0
- added U1: AMS1117-3.3, Package_TO_SOT_SMD:SOT-223-3_TabPin2, symbol Regulator_Linear:AMS1117-3.3
Connections:
- net ExVcc: now also U1.2 (VO)
- net GND: now also U1.1 (GND)
- net at J1.1: now also U1.3 (VI)
Changed lines of the file:
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@@
   (no_connect (at 127.635 71.755))
   (no_connect (at 109.855 71.755))
-  (wire (pts (xy 97.79 48.26) (xy 115.57 48.26))
-    (stroke (width 0) (type default))
-  )
   (wire (pts (xy 112.395 65.405) (xy 137.16 65.405))
     (stroke (width 0) (type default))
@@
     (stroke (width 0) (type default))
   )
+  (wire (pts (xy 87.63 48.26) (xy 87.63 40.64))
+    (stroke (width 0) (type default))
+  )
   (wire (pts (xy 118.745 71.755) (xy 117.475 71.755))
     (stroke (width 0) (type default))
@@
     (stroke (width 0) (type default))
   )
-  (wire (pts (xy 81.28 48.26) (xy 92.71 48.26))
+  (wire (pts (xy 102.87 48.26) (xy 102.87 40.64))
     (stroke (width 0) (type default))
   )
@@
     (stroke (width 0) (type default))
   )
+  (wire (pts (xy 115.57 48.26) (xy 102.87 48.26))
+    (stroke (width 0) (type default))
+  )
   (wire (pts (xy 106.68 53.975) (xy 110.49 53.975))
     (stroke (width 0) (type default))
@@
   )
   (wire (pts (xy 118.745 107.315) (xy 117.475 107.315))
+    (stroke (width 0) (type default))
+  )
+  (wire (pts (xy 81.28 48.26) (xy 87.63 48.26))
     (stroke (width 0) (type default))
   )
@@
         (path "/d5200c1e-908a-4e72-95f9-aca3b7bcc08a"
           (reference "#PWR06") (unit 1)
+        )
+      )
+    )
+  )
+  (symbol (lib_id "Regulator_Linear:AMS1117-3.3") (at 95.25 40.64 0) (unit 1)
+    (in_bom yes) (on_board yes) (dnp no) (fields_autoplaced)
+    (property "Reference" "U1" (at 95.25 34.29 0)
+      (effects (font (size 1.27 1.27)))
+    )
+    (property "Value" "AMS1117-3.3" (at 95.25 36.83 0)
+      (effects (font (size 1.27 1.27)))
+    )
+    (property "Footprint" "Package_TO_SOT_SMD:SOT-223-3_TabPin2" (at 95.25 35.56 0)
+      (effects (font (size 1.27 1.27)) hide)
+    )
+    (property "Datasheet" "http://www.advanced-monolithic.com/pdf/ds1117.pdf" (at 97.79 46.99 0)
+      (effects (font (size 1.27 1.27)) hide)
+    )
+    (pin "1")
+    (pin "2")
+    (pin "3")
+    (instances
+      (project "Pmod_PLED"
+        (path "/d5200c1e-908a-4e72-95f9-aca3b7bcc08a"
+          (reference "U1") (unit 1)
         )
       )
@@
         )
       )
-    )
-  )
-  (symbol (lib_id "SamacSys_Parts:LM2940T-5.0") (at 92.71 48.26 90) (unit 1)
-    (in_bom yes) (on_board yes) (dnp no) (fields_autoplaced)
-    (property "Reference" "IC2" (at 101.6 36.195 90)
-      (effects (font (size 1.27 1.27)) (justify right))
-    )
-    (property "Value" "LM2940T-5.0" (at 101.6 38.735 90)
-      (effects (font (size 1.27 1.27)) (justify right))
-    )
-    (property "Footprint" "SamacSys_Parts:TO254P470X1016X2222-3P" (at 90.17 29.21 0)
-      (effects (font (size 1.27 1.27)) (justify left) hide)
-    )
-    (property "Datasheet" "http://uk.rs-online.com/web/p/products/0411769" (at 92.71 29.21 0)
-      (effects (font (size 1.27 1.27)) (justify left) hide)
-    )
-    (property "Description" "IC, LDO VOLT REG, 5V, 1A" (at 95.25 29.21 0)
-      (effects (font (size 1.27 1.27)) (justify left) hide)
-    )
-    (property "Height" "" (at 97.79 29.21 0)
-      (effects (font (size 1.27 1.27)) (justify left) hide)
-    )
-    (property "RS Part Number" "0411769" (at 100.33 29.21 0)
-      (effects (font (size 1.27 1.27)) (justify left) hide)
-    )
-    (property "RS Price/Stock" "http://uk.rs-online.com/web/p/products/0411769" (at 102.87 29.21 0)
-      (effects (font (size 1.27 1.27)) (justify left) hide)
-    )
-    (property "Manufacturer_Name" "Texas Instruments" (at 105.41 29.21 0)
-      (effects (font (size 1.27 1.27)) (justify left) hide)
-    )
-    (property "Manufacturer_Part_Number" "LM2940T-5.0" (at 107.95 29.21 0)
-      (effects (font (size 1.27 1.27)) (justify left) hide)
-    )
-    (pin "1")
-    (pin "2")
-    (pin "3")
-    (instances
-      (project "Pmod_PLED"
-        (path "/d5200c1e-908a-4e72-95f9-aca3b7bcc08a"
-          (reference "IC2") (unit 1)
-        )
-      )

Commit message: 618
Parts:
- removed TP1: TestPoint, TestPoint:TestPoint_Pad_D2.0mm, symbol Connector:TestPoint
- added C1, C2: 0.1u, Capacitor_SMD:C_0603_1608Metric_Pad1.08x0.95mm_HandSolder, symbol Device:C
Connections:
- net ExVcc: now also C2.2
- net GND: now also C1.2, C2.1
- net at D1.2 (RK): now also IC1.16 (O4); no longer IC1.7 (O2)
- net at J1.1, U1.3 (VI): now also C1.1
Changed lines of the file:
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@@
 (kicad_sch (version 20230121) (generator eeschema)
   (paper "A4")
+  (junction (at 102.87 48.26) (diameter 0) (color 0 0 0 0)
+  )
+  (junction (at 87.63 48.26) (diameter 0) (color 0 0 0 0)
+  )
   (junction (at 95.25 53.34) (diameter 0) (color 0 0 0 0)
+  )
+  (junction (at 95.25 48.26) (diameter 0) (color 0 0 0 0)
   )
   (junction (at 118.745 107.315) (diameter 0) (color 0 0 0 0)
@@
   (no_connect (at 127.635 71.755))
   (no_connect (at 109.855 71.755))
-  (wire (pts (xy 112.395 65.405) (xy 137.16 65.405))
+  (wire (pts (xy 137.16 81.915) (xy 137.16 107.315))
     (stroke (width 0) (type default))
   )
@@
     (stroke (width 0) (type default))
   )
-  (wire (pts (xy 127.635 107.315) (xy 130.81 107.315))
-    (stroke (width 0) (type default))
-  )
   (wire (pts (xy 137.16 81.915) (xy 142.875 81.915))
     (stroke (width 0) (type default))
@@
     (stroke (width 0) (type default))
   )
-  (wire (pts (xy 137.16 65.405) (xy 137.16 81.915))
-    (stroke (width 0) (type default))
-  )
   (wire (pts (xy 86.36 62.865) (xy 122.555 62.865))
     (stroke (width 0) (type default))
@@
     (stroke (width 0) (type default))
   )
-  (wire (pts (xy 112.395 65.405) (xy 112.395 71.755))
+  (wire (pts (xy 137.16 107.315) (xy 127.635 107.315))
     (stroke (width 0) (type default))
   )
@@
     )
   )
-  (symbol (lib_id "Connector:TestPoint") (at 130.81 107.315 0) (unit 1)
-    (in_bom yes) (on_board yes) (dnp no) (fields_autoplaced)
-    (property "Reference" "TP1" (at 133.35 103.378 0)
-      (effects (font (size 1.27 1.27)) (justify left))
-    )
-    (property "Value" "TestPoint" (at 133.35 105.918 0)
-      (effects (font (size 1.27 1.27)) (justify left))
-    )
-    (property "Footprint" "TestPoint:TestPoint_Pad_D2.0mm" (at 135.89 107.315 0)
-      (effects (font (size 1.27 1.27)) hide)
-    )
-    (property "Datasheet" "~" (at 135.89 107.315 0)
-      (effects (font (size 1.27 1.27)) hide)
-    )
-    (pin "1")
-    (instances
-      (project "Pmod_PLED"
-        (path "/d5200c1e-908a-4e72-95f9-aca3b7bcc08a"
-          (reference "TP1") (unit 1)
+  (symbol (lib_id "Device:C") (at 91.44 48.26 90) (unit 1)
+    (in_bom yes) (on_board yes) (dnp no) (fields_autoplaced)
+    (property "Reference" "C1" (at 91.44 41.91 90)
+      (effects (font (size 1.27 1.27)))
+    )
+    (property "Value" "0.1u" (at 91.44 44.45 90)
+      (effects (font (size 1.27 1.27)))
+    )
+    (property "Footprint" "Capacitor_SMD:C_0603_1608Metric_Pad1.08x0.95mm_HandSolder" (at 95.25 47.2948 0)
+      (effects (font (size 1.27 1.27)) hide)
+    )
+    (property "Datasheet" "~" (at 91.44 48.26 0)
+      (effects (font (size 1.27 1.27)) hide)
+    )
+    (pin "1")
+    (pin "2")
+    (instances
+      (project "Pmod_PLED"
+        (path "/d5200c1e-908a-4e72-95f9-aca3b7bcc08a"
+          (reference "C1") (unit 1)
         )
       )
@@
         )
       )
+    )
+  )
+  (symbol (lib_id "Device:C") (at 99.06 48.26 90) (unit 1)
+    (in_bom yes) (on_board yes) (dnp no) (fields_autoplaced)
+    (property "Reference" "C2" (at 99.06 41.91 90)
+      (effects (font (size 1.27 1.27)))
+    )
+    (property "Value" "0.1u" (at 99.06 44.45 90)
+      (effects (font (size 1.27 1.27)))
+    )
+    (property "Footprint" "Capacitor_SMD:C_0603_1608Metric_Pad1.08x0.95mm_HandSolder" (at 102.87 47.2948 0)
+      (effects (font (size 1.27 1.27)) hide)
+    )
+    (property "Datasheet" "~" (at 99.06 48.26 0)
+      (effects (font (size 1.27 1.27)) hide)
+    )
+    (pin "1")
+    (pin "2")
+    (instances
+      (project "Pmod_PLED"
+        (path "/d5200c1e-908a-4e72-95f9-aca3b7bcc08a"
+          (reference "C2") (unit 1)
+        )
+      )
