File: Pmod_PLED/kikit/PmodPLED_kikit.kicad_pcb (KiCad board)
At the start: 2 copper layers, 88.5 x 101.3 mm, 212 parts, among them IC1 TBD62064APG, IC2 LM2940T-5.0, J1 Barrel_Jack_Switch, J3 Conn_01x03_Pin

Commit message: 601
Parts:
- removed the D1 at (151.2, 104.3)
- removed the D1 at (151.2, 37.3)
- removed the D1 at (151.2, 59.7)
- removed the D1 at (151.2, 82.0)
- removed the D3 at (161.6, 45.2)
- removed the D3 at (161.6, 112.1)
- removed the D3 at (161.6, 89.8)
- removed the D3 at (161.6, 67.5)
- removed the IC1 at (127.5, 33.2)
- removed the IC1 at (127.5, 77.9)
- removed the IC1 at (127.5, 100.2)
- removed the IC1 at (127.5, 55.5)
- removed the IC2 at (183.7, 57.2)
- removed the IC2 at (183.7, 34.9)
- removed the IC2 at (183.7, 79.5)
- removed the IC2 at (183.7, 101.8)
- removed the J1 at (171.8, 42.5)
- removed the J1 at (171.8, 87.1)
- removed the J1 at (171.8, 109.5)
- removed the J1 at (171.8, 64.8)
- removed the J3 at (156.9, 96.2)
- removed the J3 at (156.9, 29.3)
- removed the J3 at (156.9, 73.9)
- removed the J3 at (156.9, 51.6)
- removed the REF** at (147.6, 47.3)
- removed the REF** at (111.3, 105.9)
- removed the REF** at (148.5, 47.3)
- removed the REF** at (111.3, 36.3)
- removed the REF** at (185.7, 58.6)
- removed the REF** at (147.6, 71.6)
- removed the REF** at (111.3, 63.0)
- removed the REF** at (150.2, 94.0)
- removed the REF** at (149.4, 92.0)
- removed the REF** at (185.7, 104.1)
- removed the REF** at (147.6, 49.3)
- removed the REF** at (145.0, 49.3)
- removed the REF** at (151.1, 71.6)
- removed the REF** at (145.0, 114.3)
- removed the REF** at (152.0, 71.6)
- removed the REF** at (111.3, 23.4)
- removed the REF** at (148.5, 94.0)
- removed the REF** at (192.0, 114.3)
- removed the REF** at (147.6, 94.0)
- removed the REF** at (185.7, 80.9)
- removed the REF** at (111.3, 33.7)
- removed the REF** at (148.5, 49.3)
- removed the REF** at (185.7, 85.3)
- removed the REF** at (145.9, 47.3)
- removed the REF** at (185.7, 84.4)
- removed the REF** at (111.3, 80.9)
- removed the REF** at (107.6, 114.3)
- removed the REF** at (190.2, 27.0)
- removed the REF** at (185.7, 81.8)
- removed the REF** at (111.3, 82.7)
- removed the REF** at (150.2, 27.0)
- removed the REF** at (152.0, 114.3)
- removed the REF** at (185.7, 118.8)
- removed the REF** at (145.0, 27.0)
- removed the REF** at (111.3, 118.8)
- removed the REF** at (150.2, 114.3)
- removed the REF** at (185.7, 119.6)
- removed the REF** at (145.0, 69.6)
- removed the REF** at (111.3, 79.2)
- removed the REF** at (146.8, 47.3)
- removed the REF** at (185.7, 20.8)
- removed the REF** at (185.7, 117.9)
- removed the REF** at (185.7, 38.9)
- removed the REF** at (189.4, 114.3)
- removed the REF** at (185.7, 103.2)
- removed the REF** at (185.7, 100.6)
- removed the REF** at (111.3, 57.7)
- removed the REF** at (185.7, 61.2)
- removed the REF** at (111.3, 62.1)
- removed the REF** at (152.0, 69.6)
- removed the REF** at (145.9, 94.0)
- removed the REF** at (146.8, 94.0)
- removed the REF** at (150.2, 71.6)
- removed the REF** at (152.0, 94.0)
- removed the REF** at (111.3, 21.6)
- removed the REF** at (145.9, 49.3)
- removed the REF** at (111.3, 102.4)
- removed the REF** at (111.3, 81.8)
- removed the REF** at (152.0, 27.0)
- removed the REF** at (111.3, 84.4)
- removed the REF** at (111.3, 101.5)
- removed the REF** at (147.6, 114.3)
- removed the REF** at (145.0, 94.0)
- removed the REF** at (111.3, 38.0)
- removed the REF** at (111.3, 24.2)
- removed the REF** at (191.1, 114.3)
- removed the REF** at (147.6, 92.0)
- removed the REF** at (188.5, 27.0)
- removed the REF** at (146.8, 49.3)
- removed the REF** at (111.3, 56.0)
- removed the REF** at (145.0, 47.3)
- removed the REF** at (111.3, 38.9)
- removed the REF** at (150.2, 69.6)
- removed the REF** at (185.7, 38.0)
- removed the REF** at (146.8, 92.0)
- removed the REF** at (185.7, 57.7)
- removed the REF** at (148.5, 92.0)
- removed the REF** at (185.7, 23.4)
- removed the REF** at (185.7, 107.6)
- removed the REF** at (149.4, 49.3)
- removed the REF** at (185.7, 35.4)
- removed the REF** at (185.7, 83.5)
- removed the REF** at (152.0, 92.0)
- removed the REF** at (111.3, 34.5)
- removed the REF** at (111.3, 39.8)
- removed the REF** at (185.7, 33.7)
- removed the REF** at (148.5, 69.6)
- removed the REF** at (151.1, 94.0)
- removed the REF** at (149.4, 69.6)
- removed the REF** at (147.6, 69.6)
- removed the REF** at (149.4, 71.6)
- removed the REF** at (185.7, 101.5)
- removed the REF** at (185.7, 21.6)
- removed the REF** at (146.8, 71.6)
- removed the REF** at (106.8, 27.0)
- removed the REF** at (151.1, 49.3)
- removed the REF** at (151.1, 47.3)
- removed the REF** at (185.7, 80.0)
- removed the REF** at (111.3, 107.6)
- removed the REF** at (146.8, 27.0)
- removed the REF** at (185.7, 39.8)
- removed the REF** at (149.4, 27.0)
- removed the REF** at (150.2, 92.0)
- removed the REF** at (111.3, 78.3)
- removed the REF** at (111.3, 60.4)
- removed the REF** at (111.3, 117.9)
- removed the REF** at (105.0, 27.0)
- removed the REF** at (111.3, 20.8)
- removed the REF** at (145.9, 114.3)
- removed the REF** at (185.7, 105.0)
- removed the REF** at (185.7, 40.7)
- removed the REF** at (145.9, 71.6)
- removed the REF** at (145.9, 69.6)
- removed the REF** at (148.5, 27.0)
- removed the REF** at (185.7, 106.7)
- removed the REF** at (145.0, 92.0)
- removed the REF** at (111.3, 106.7)
- removed the REF** at (190.2, 114.3)
- removed the REF** at (192.0, 27.0)
- removed the REF** at (189.4, 27.0)
- removed the REF** at (188.5, 114.3)
- removed the REF** at (185.7, 117.0)
- removed the REF** at (191.1, 27.0)
- removed the REF** at (185.7, 60.4)
- removed the REF** at (185.7, 22.5)
- removed the REF** at (149.4, 47.3)
- removed the REF** at (111.3, 37.2)
- removed the REF** at (185.7, 79.2)
- removed the REF** at (148.5, 114.3)
- removed the REF** at (185.7, 56.9)
- removed the REF** at (150.2, 49.3)
- removed the REF** at (185.7, 102.4)
- removed the REF** at (185.7, 62.1)
- removed the REF** at (185.7, 34.5)
- removed the REF** at (105.9, 27.0)
- removed the REF** at (150.2, 47.3)
- removed the REF** at (111.3, 104.1)
- removed the REF** at (149.4, 94.0)
- removed the REF** at (105.0, 114.3)
- removed the REF** at (147.6, 27.0)
- removed the REF** at (185.7, 24.2)
- removed the REF** at (185.7, 56.0)
- removed the REF** at (111.3, 35.4)
- removed the REF** at (108.5, 114.3)
- removed the REF** at (106.8, 114.3)
- removed the REF** at (105.9, 114.3)
- removed the REF** at (152.0, 49.3)
- removed the REF** at (111.3, 85.3)
- removed the REF** at (185.7, 36.3)
- removed the REF** at (185.7, 63.0)
- removed the REF** at (111.3, 59.5)
- removed the REF** at (107.6, 27.0)
- removed the REF** at (111.3, 40.7)
- removed the REF** at (185.7, 82.7)
- removed the REF** at (185.7, 105.9)
- removed the REF** at (146.8, 69.6)
- removed the REF** at (152.0, 47.3)
- removed the REF** at (111.3, 83.5)
- removed the REF** at (111.3, 100.6)
- removed the REF** at (111.3, 103.2)
- removed the REF** at (148.5, 71.6)
- removed the REF** at (111.3, 56.9)
- removed the REF** at (151.1, 114.3)
- removed the REF** at (185.7, 120.5)
- removed the REF** at (108.5, 27.0)
- removed the REF** at (111.3, 119.6)
- removed the REF** at (185.7, 78.3)
- removed the REF** at (145.0, 71.6)
- removed the REF** at (145.9, 27.0)
- removed the REF** at (146.8, 114.3)
- removed the REF** at (185.7, 37.2)
- removed the REF** at (145.9, 92.0)
- removed the REF** at (111.3, 22.5)
- removed the REF** at (111.3, 117.0)
- removed the REF** at (111.3, 120.5)
- removed the REF** at (111.3, 105.0)
- removed the REF** at (151.1, 27.0)
- removed the REF** at (111.3, 58.6)
- removed the REF** at (149.4, 114.3)
- removed the REF** at (185.7, 59.5)
- removed the REF** at (151.1, 92.0)
- removed the REF** at (111.3, 80.0)
- removed the REF** at (111.3, 61.2)
- removed the REF** at (151.1, 69.6)
- removed the Reserve at (135.1, 107.6)
- removed the Reserve at (135.1, 62.9)
- removed the Reserve at (135.1, 85.2)
- removed the Reserve at (135.1, 40.6)
- added D1: [EP204K-150G1R1B1-CA], MyLibrary:EP204-150G1R1B1-CA, F.Cu at (151.2, 58.7)
- added D1: [EP204K-150G1R1B1-CA], MyLibrary:EP204-150G1R1B1-CA, F.Cu at (151.2, 103.3)
- added D1: [EP204K-150G1R1B1-CA], MyLibrary:EP204-150G1R1B1-CA, F.Cu at (151.2, 81.0)
- added D1: [EP204K-150G1R1B1-CA], MyLibrary:EP204-150G1R1B1-CA, F.Cu at (151.2, 36.3)
- added D3: SS2040FL, SamacSys_Parts:SODFL3618X108N, F.Cu at (161.6, 66.5)
- added D3: SS2040FL, SamacSys_Parts:SODFL3618X108N, F.Cu at (161.6, 111.1)
- added D3: SS2040FL, SamacSys_Parts:SODFL3618X108N, F.Cu at (161.6, 88.8)
- added D3: SS2040FL, SamacSys_Parts:SODFL3618X108N, F.Cu at (161.6, 44.2)
- added G***: LOGO, MyLibrary:logo_kamo_ss, F.Cu at (175.4, 97.3)
- added G***: LOGO, MyLibrary:logo_kamo_ss, F.Cu at (175.4, 30.3)
- added G***: LOGO, MyLibrary:logo_kamo_ss, F.Cu at (175.4, 75.0)
- added G***: LOGO, MyLibrary:logo_kamo_ss, F.Cu at (175.4, 52.6)
- added IC1: TBD62064APG, SamacSys_Parts:DIP762W60P254L1975H445Q16N, F.Cu at (127.5, 76.9)
- added IC1: TBD62064APG, SamacSys_Parts:DIP762W60P254L1975H445Q16N, F.Cu at (127.5, 99.2)
- added IC1: TBD62064APG, SamacSys_Parts:DIP762W60P254L1975H445Q16N, F.Cu at (127.5, 54.5)
- added IC1: TBD62064APG, SamacSys_Parts:DIP762W60P254L1975H445Q16N, F.Cu at (127.5, 32.2)
- added IC2: LM2940T-5.0, SamacSys_Parts:TO254P470X1016X2222-3P, F.Cu at (182.7, 73.6)
- added IC2: LM2940T-5.0, SamacSys_Parts:TO254P470X1016X2222-3P, F.Cu at (182.7, 28.9)
- added IC2: LM2940T-5.0, SamacSys_Parts:TO254P470X1016X2222-3P, F.Cu at (182.7, 51.2)
- added IC2: LM2940T-5.0, SamacSys_Parts:TO254P470X1016X2222-3P, F.Cu at (182.7, 95.9)
- added J1: Barrel_Jack_Switch, Connector_BarrelJack:BarrelJack_Horizontal, F.Cu at (171.8, 86.5)
- added J1: Barrel_Jack_Switch, Connector_BarrelJack:BarrelJack_Horizontal, F.Cu at (171.8, 108.8)
- added J1: Barrel_Jack_Switch, Connector_BarrelJack:BarrelJack_Horizontal, F.Cu at (171.8, 64.1)
- added J1: Barrel_Jack_Switch, Connector_BarrelJack:BarrelJack_Horizontal, F.Cu at (171.8, 41.8)
- added J2: Conn_01x06_Pin, Library:Pmod6, F.Cu at (111.4, 28.5)
- added J2: Conn_01x06_Pin, Library:Pmod6, F.Cu at (111.4, 73.2)
- added J2: Conn_01x06_Pin, Library:Pmod6, F.Cu at (111.4, 50.9)
- added J2: Conn_01x06_Pin, Library:Pmod6, F.Cu at (111.4, 95.5)
- added J3: Conn_01x03_Pin, Connector_PinHeader_2.54mm:PinHeader_1x03_P2.54mm_Vertical, F.Cu at (156.9, 72.9)
- added J3: Conn_01x03_Pin, Connector_PinHeader_2.54mm:PinHeader_1x03_P2.54mm_Vertical, F.Cu at (156.9, 50.6)
- added J3: Conn_01x03_Pin, Connector_PinHeader_2.54mm:PinHeader_1x03_P2.54mm_Vertical, F.Cu at (156.9, 28.3)
- added J3: Conn_01x03_Pin, Connector_PinHeader_2.54mm:PinHeader_1x03_P2.54mm_Vertical, F.Cu at (156.9, 95.2)
- added REF**: NPTH, NPTH, F.Cu at (111.0, 103.1)
- added REF**: NPTH, NPTH, F.Cu at (149.4, 48.1)
- added REF**: NPTH, NPTH, F.Cu at (186.0, 57.6)
- added REF**: NPTH, NPTH, F.Cu at (150.2, 70.4)
- added REF**: NPTH, NPTH, F.Cu at (190.2, 113.3)
- added REF**: NPTH, NPTH, F.Cu at (111.0, 37.9)
- added REF**: NPTH, NPTH, F.Cu at (191.0, 113.3)
- added REF**: NPTH, NPTH, F.Cu at (186.0, 80.8)
- added REF**: NPTH, NPTH, F.Cu at (147.6, 48.1)
- added REF**: NPTH, NPTH, F.Cu at (111.3, 116.8)
- added REF**: NPTH, NPTH, F.Cu at (188.4, 113.3)
- added REF**: NPTH, NPTH, F.Cu at (146.8, 113.5)
- added REF**: NPTH, NPTH, F.Cu at (111.0, 34.4)
- added REF**: NPTH, NPTH, F.Cu at (186.0, 82.5)
- added REF**: NPTH, NPTH, F.Cu at (147.6, 91.2)
- added REF**: NPTH, NPTH, F.Cu at (106.0, 26.0)
- added REF**: NPTH, NPTH, F.Cu at (150.2, 113.5)
- added REF**: NPTH, NPTH, F.Cu at (146.8, 68.9)
- added REF**: NPTH, NPTH, F.Cu at (186.0, 34.4)
- added REF**: NPTH, NPTH, F.Cu at (150.2, 25.8)
- added REF**: NPTH, NPTH, F.Cu at (148.5, 113.5)
- added REF**: NPTH, NPTH, F.Cu at (186.0, 104.0)
- added REF**: NPTH, NPTH, F.Cu at (185.7, 116.8)
- added REF**: NPTH, NPTH, F.Cu at (149.4, 25.8)
- added REF**: NPTH, NPTH, F.Cu at (106.0, 113.3)
- added REF**: NPTH, NPTH, F.Cu at (186.0, 36.2)
- added REF**: NPTH, NPTH, F.Cu at (111.0, 81.7)
- added REF**: NPTH, NPTH, F.Cu at (149.4, 70.4)
- added REF**: NPTH, NPTH, F.Cu at (111.0, 59.4)
- added REF**: NPTH, NPTH, F.Cu at (111.0, 35.3)
- added REF**: NPTH, NPTH, F.Cu at (189.3, 26.0)
- added REF**: NPTH, NPTH, F.Cu at (111.0, 60.2)
- added REF**: NPTH, NPTH, F.Cu at (108.6, 26.0)
- added REF**: NPTH, NPTH, F.Cu at (111.0, 37.0)
- added REF**: NPTH, NPTH, F.Cu at (186.0, 101.4)
- added REF**: NPTH, NPTH, F.Cu at (186.0, 102.2)
- added REF**: NPTH, NPTH, F.Cu at (186.0, 79.9)
- added REF**: NPTH, NPTH, F.Cu at (150.2, 68.9)
- added REF**: NPTH, NPTH, F.Cu at (111.0, 79.9)
- added REF**: NPTH, NPTH, F.Cu at (149.4, 92.7)
- added REF**: NPTH, NPTH, F.Cu at (191.0, 26.0)
- added REF**: NPTH, NPTH, F.Cu at (150.2, 91.2)
- added REF**: NPTH, NPTH, F.Cu at (188.4, 26.0)
- added REF**: NPTH, NPTH, F.Cu at (190.2, 26.0)
- added REF**: NPTH, NPTH, F.Cu at (150.2, 92.7)
- added REF**: NPTH, NPTH, F.Cu at (111.0, 104.9)
- added REF**: NPTH, NPTH, F.Cu at (111.3, 117.7)
- added REF**: NPTH, NPTH, F.Cu at (146.8, 46.6)
- added REF**: NPTH, NPTH, F.Cu at (111.0, 82.5)
- added REF**: NPTH, NPTH, F.Cu at (186.0, 79.0)
- added REF**: NPTH, NPTH, F.Cu at (146.8, 48.1)
- added REF**: NPTH, NPTH, F.Cu at (185.7, 117.7)
- added REF**: NPTH, NPTH, F.Cu at (148.5, 68.9)
- added REF**: NPTH, NPTH, F.Cu at (148.5, 25.8)
- added REF**: NPTH, NPTH, F.Cu at (146.8, 25.8)
- added REF**: NPTH, NPTH, F.Cu at (106.8, 26.0)
- added REF**: NPTH, NPTH, F.Cu at (149.4, 91.2)
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Routing:
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Other:
- board size 88.5 x 101.3 mm -> 86.5 x 99.3 mm

Commit message: 601b
Parts:
- removed the IC1 at (127.5, 76.9)
- removed the IC1 at (127.5, 99.2)
- removed the IC1 at (127.5, 54.5)
- removed the IC1 at (127.5, 32.2)
- removed Reserve (x4): TestPoint, TestPoint:TestPoint_Pad_D2.0mm
- added IC1: TBD62064APG, SamacSys_Parts:DIP762W60P254L1975H445Q16N, F.Cu at (127.5, 57.9)
- added IC1: TBD62064APG, SamacSys_Parts:DIP762W60P254L1975H445Q16N, F.Cu at (127.5, 80.2)
- added IC1: TBD62064APG, SamacSys_Parts:DIP762W60P254L1975H445Q16N, F.Cu at (127.5, 102.5)
- added IC1: TBD62064APG, SamacSys_Parts:DIP762W60P254L1975H445Q16N, F.Cu at (127.5, 35.5)
- added TP1: TestPoint, TestPoint:TestPoint_Pad_D2.0mm, F.Cu at (135.1, 42.0)
- added TP1: TestPoint, TestPoint:TestPoint_Pad_D2.0mm, F.Cu at (135.1, 64.3)
- added TP1: TestPoint, TestPoint:TestPoint_Pad_D2.0mm, F.Cu at (135.1, 86.6)
- added TP1: TestPoint, TestPoint:TestPoint_Pad_D2.0mm, F.Cu at (135.1, 109.0)
- D1 (x4): value [EP204K-150G1R1B1-CA] -> EP204K-150G1R1B1-CA
Connections:
- D1 pad 5: Board_0-Net-(IC1-O2) -> Board_0-unconnected-(D1-RK-Pad5)
- D1 pad 5: Board_2-Net-(IC1-O2) -> Board_2-unconnected-(D1-RK-Pad5)
- D1 pad 5: Board_3-Net-(IC1-O2) -> Board_3-unconnected-(D1-RK-Pad5)
- D1 pad 5: Board_1-Net-(IC1-O2) -> Board_1-unconnected-(D1-RK-Pad5)
Routing:
- net Board_2-Net-(IC1-O2): track 39.4 -> 21.8 mm
- net Board_0-Net-(IC1-O2): track 39.4 -> 21.8 mm
- net Board_1-Net-(IC1-O2): track 39.4 -> 21.8 mm
- net Board_3-Net-(IC1-O2): track 39.4 -> 21.8 mm
- net Board_2-VCC: track 52.4 -> 62.2 mm
- net Board_3-VCC: track 52.4 -> 62.2 mm
- net Board_1-VCC: track 52.4 -> 62.2 mm
- net Board_0-VCC: track 52.4 -> 62.2 mm
- net Board_3-Net-(IC1-I1): track 19.3 -> 18.0 mm
- net Board_1-Net-(IC1-I1): track 19.3 -> 18.0 mm
- net Board_0-Net-(IC1-I1): track 19.3 -> 18.0 mm
- net Board_2-Net-(IC1-I1): track 19.3 -> 18.0 mm
- net Board_2-Net-(IC1-O4): track 4.08 -> 3.19 mm
- net Board_1-Net-(IC1-O4): track 4.08 -> 3.19 mm
- net Board_0-Net-(IC1-O4): track 4.08 -> 3.19 mm
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- removed copper zone on B.Cu, net Board_0-GND
- removed copper zone on B.Cu, net Board_1-GND
- removed copper zone on B.Cu, net Board_2-GND
- removed copper zone on B.Cu, net Board_3-GND

Commit message: 601c
Parts:
- removed the G*** at (175.4, 52.6)
- removed the G*** at (175.4, 75.0)
- removed the G*** at (175.4, 30.3)
- removed the G*** at (175.4, 97.3)
- removed TP1 (x4): TestPoint, TestPoint:TestPoint_Pad_D2.0mm
- added G***: LOGO, MyLibrary:logo_kamo_ss, F.Cu at (175.4, 97.4)
- added G***: LOGO, MyLibrary:logo_kamo_ss, F.Cu at (175.4, 75.1)
- added G***: LOGO, MyLibrary:logo_kamo_ss, F.Cu at (175.4, 30.5)
- added G***: LOGO, MyLibrary:logo_kamo_ss, F.Cu at (175.4, 52.8)
- added Reserve: TestPoint, TestPoint:TestPoint_Pad_D2.0mm, F.Cu at (135.1, 109.0)
- added Reserve: TestPoint, TestPoint:TestPoint_Pad_D2.0mm, F.Cu at (135.1, 64.3)
- added Reserve: TestPoint, TestPoint:TestPoint_Pad_D2.0mm, F.Cu at (135.1, 86.6)
- added Reserve: TestPoint, TestPoint:TestPoint_Pad_D2.0mm, F.Cu at (135.1, 42.0)
Other:
- board text added: "ExVcc"
- board text removed: "Ex Vcc"

Commit message: 601d
Parts:
- removed the D1 at (151.2, 36.3)
- removed the D1 at (151.2, 103.3)
- removed the D1 at (151.2, 81.0)
- removed the D1 at (151.2, 58.7)
- removed the D3 at (161.6, 66.5)
- removed the D3 at (161.6, 111.1)
- removed the D3 at (161.6, 88.8)
- removed the D3 at (161.6, 44.2)
- removed the G*** at (175.4, 97.4)
- removed the G*** at (175.4, 75.1)
- removed the G*** at (175.4, 30.5)
- removed the G*** at (175.4, 52.8)
- removed the IC1 at (127.5, 80.2)
- removed the IC1 at (127.5, 35.5)
- removed the IC1 at (127.5, 102.5)
- removed the IC1 at (127.5, 57.9)
- removed the IC2 at (182.7, 95.9)
- removed the IC2 at (182.7, 51.2)
- removed the IC2 at (182.7, 28.9)
- removed the IC2 at (182.7, 73.6)
- removed the J1 at (171.8, 64.1)
- removed the J1 at (171.8, 86.5)
- removed the J1 at (171.8, 108.8)
- removed the J1 at (171.8, 41.8)
- removed the J2 at (111.4, 95.5)
- removed the J2 at (111.4, 73.2)
- removed the J2 at (111.4, 50.9)
- removed the J2 at (111.4, 28.5)
- removed the J3 at (156.9, 28.3)
- removed the J3 at (156.9, 72.9)
- removed the J3 at (156.9, 95.2)
- removed the J3 at (156.9, 50.6)
- removed the REF** at (111.0, 35.3)
- removed the REF** at (186.0, 103.1)
- removed the REF** at (147.6, 70.4)
- removed the REF** at (111.3, 118.6)
- removed the REF** at (150.2, 46.6)
- removed the REF** at (185.7, 118.6)
- removed the REF** at (111.0, 60.2)
- removed the REF** at (111.3, 116.8)
- removed the REF** at (189.3, 113.3)
- removed the REF** at (106.8, 26.0)
- removed the REF** at (149.4, 48.1)
- removed the REF** at (108.6, 113.3)
- removed the REF** at (111.0, 37.0)
- removed the REF** at (186.0, 60.2)
- removed the REF** at (150.2, 92.7)
- removed the REF** at (186.0, 56.7)
- removed the REF** at (150.2, 113.5)
- removed the REF** at (185.7, 23.3)
- removed the REF** at (111.0, 82.5)
- removed the REF** at (108.6, 26.0)
- removed the REF** at (111.0, 102.2)
- removed the REF** at (111.0, 57.6)
- removed the REF** at (147.6, 25.8)
- removed the REF** at (146.8, 70.4)
- removed the REF** at (186.0, 37.9)
- removed the REF** at (189.3, 26.0)
- removed the REF** at (146.8, 25.8)
- removed the REF** at (111.3, 22.4)
- removed the REF** at (107.7, 26.0)
- removed the REF** at (111.3, 23.3)
- removed the REF** at (186.0, 79.0)
- removed the REF** at (111.0, 81.7)
- removed the REF** at (186.0, 59.4)
- removed the REF** at (106.8, 113.3)
- removed the REF** at (185.7, 116.0)
- removed the REF** at (149.4, 70.4)
- removed the REF** at (185.7, 117.7)
- removed the REF** at (148.5, 46.6)
- removed the REF** at (147.6, 48.1)
- removed the REF** at (186.0, 58.5)
- removed the REF** at (111.3, 20.7)
- removed the REF** at (111.0, 79.0)
- removed the REF** at (186.0, 101.4)
- removed the REF** at (111.0, 59.4)
- removed the REF** at (148.5, 113.5)
- removed the REF** at (186.0, 80.8)
- removed the REF** at (186.0, 102.2)
- removed the REF** at (185.7, 20.7)
- removed the REF** at (186.0, 36.2)
- removed the REF** at (146.8, 68.9)
- removed the REF** at (186.0, 104.0)
- removed the REF** at (149.4, 46.6)
- removed the REF** at (147.6, 68.9)
- removed the REF** at (148.5, 91.2)
- removed the REF** at (149.4, 91.2)
- removed the REF** at (185.7, 22.4)
- removed the REF** at (186.0, 37.0)
- removed the REF** at (186.0, 81.7)
- removed the REF** at (106.0, 26.0)
- removed the REF** at (147.6, 91.2)
- removed the REF** at (146.8, 91.2)
- removed the REF** at (186.0, 34.4)
- removed the REF** at (111.3, 117.7)
- removed the REF** at (111.0, 37.9)
- removed the REF** at (191.0, 113.3)
- removed the REF** at (188.4, 26.0)
- removed the REF** at (190.2, 26.0)
- removed the REF** at (146.8, 92.7)
- removed the REF** at (148.5, 25.8)
- removed the REF** at (147.6, 92.7)
- removed the REF** at (185.7, 21.6)
- removed the REF** at (186.0, 82.5)
- removed the REF** at (150.2, 70.4)
- removed the REF** at (111.3, 116.0)
- removed the REF** at (146.8, 48.1)
- removed the REF** at (106.0, 113.3)
- removed the REF** at (107.7, 113.3)
- removed the REF** at (111.3, 21.6)
- removed the REF** at (111.0, 34.4)
- removed the REF** at (190.2, 113.3)
- removed the REF** at (147.6, 113.5)
- removed the REF** at (185.7, 116.8)
- removed the REF** at (148.5, 48.1)
- removed the REF** at (191.0, 26.0)
- removed the REF** at (111.0, 36.2)
- removed the REF** at (186.0, 79.9)
- removed the REF** at (186.0, 57.6)
- removed the REF** at (111.0, 80.8)
- removed the REF** at (186.0, 35.3)
- removed the REF** at (147.6, 46.6)
- removed the REF** at (146.8, 46.6)
- removed the REF** at (146.8, 113.5)
- removed the REF** at (111.0, 56.7)
- removed the REF** at (111.0, 58.5)
- removed the REF** at (111.0, 104.9)
- removed the REF** at (150.2, 68.9)
- removed the REF** at (150.2, 48.1)
- removed the REF** at (148.5, 70.4)
- removed the REF** at (149.4, 92.7)
- removed the REF** at (111.0, 103.1)
- removed the REF** at (111.0, 101.4)
- removed the REF** at (149.4, 68.9)
- removed the REF** at (111.0, 104.0)
- removed the REF** at (188.4, 113.3)
- removed the REF** at (186.0, 104.9)
- removed the REF** at (111.0, 79.9)
- removed the REF** at (149.4, 25.8)
- removed the REF** at (150.2, 25.8)
- removed the REF** at (148.5, 68.9)
- removed the REF** at (148.5, 92.7)
- removed the REF** at (149.4, 113.5)
- removed the REF** at (150.2, 91.2)
- removed the Reserve at (135.1, 109.0)
- removed the Reserve at (135.1, 64.3)
- removed the Reserve at (135.1, 86.6)
- removed the Reserve at (135.1, 42.0)
- added D1: EP204K-150G1R1B1-CA, MyLibrary:EP204-150G1R1B1-CA, F.Cu at (151.2, 102.9)
- added D1: EP204K-150G1R1B1-CA, MyLibrary:EP204-150G1R1B1-CA, F.Cu at (151.2, 35.3)
- added D1: EP204K-150G1R1B1-CA, MyLibrary:EP204-150G1R1B1-CA, F.Cu at (151.2, 57.9)
- added D1: EP204K-150G1R1B1-CA, MyLibrary:EP204-150G1R1B1-CA, F.Cu at (151.2, 80.4)
- added D3: SS2040FL, SamacSys_Parts:SODFL3618X108N, F.Cu at (161.6, 110.7)
- added D3: SS2040FL, SamacSys_Parts:SODFL3618X108N, F.Cu at (161.6, 43.2)
- added D3: SS2040FL, SamacSys_Parts:SODFL3618X108N, F.Cu at (161.6, 88.2)
- added D3: SS2040FL, SamacSys_Parts:SODFL3618X108N, F.Cu at (161.6, 65.7)
- added G***: LOGO, MyLibrary:logo_kamo_ss, F.Cu at (175.4, 74.5)
- added G***: LOGO, MyLibrary:logo_kamo_ss, F.Cu at (175.4, 97.0)
- added G***: LOGO, MyLibrary:logo_kamo_ss, F.Cu at (175.4, 52.0)
- added G***: LOGO, MyLibrary:logo_kamo_ss, F.Cu at (175.4, 29.5)
- added IC1: TBD62064APG, SamacSys_Parts:DIP762W60P254L1975H445Q16N, F.Cu at (127.5, 34.5)
- added IC1: TBD62064APG, SamacSys_Parts:DIP762W60P254L1975H445Q16N, F.Cu at (127.5, 79.6)
- added IC1: TBD62064APG, SamacSys_Parts:DIP762W60P254L1975H445Q16N, F.Cu at (127.5, 57.1)
- added IC1: TBD62064APG, SamacSys_Parts:DIP762W60P254L1975H445Q16N, F.Cu at (127.5, 102.1)
- added IC2: LM2940T-5.0, SamacSys_Parts:TO254P470X1016X2222-3P, F.Cu at (182.7, 95.5)
- added IC2: LM2940T-5.0, SamacSys_Parts:TO254P470X1016X2222-3P, F.Cu at (182.7, 50.4)
- added IC2: LM2940T-5.0, SamacSys_Parts:TO254P470X1016X2222-3P, F.Cu at (182.7, 27.9)
- added IC2: LM2940T-5.0, SamacSys_Parts:TO254P470X1016X2222-3P, F.Cu at (182.7, 73.0)
- added J1: Barrel_Jack_Switch, Connector_BarrelJack:BarrelJack_Horizontal, F.Cu at (171.8, 63.3)
- added J1: Barrel_Jack_Switch, Connector_BarrelJack:BarrelJack_Horizontal, F.Cu at (171.8, 108.4)
- added J1: Barrel_Jack_Switch, Connector_BarrelJack:BarrelJack_Horizontal, F.Cu at (171.8, 85.9)
- added J1: Barrel_Jack_Switch, Connector_BarrelJack:BarrelJack_Horizontal, F.Cu at (171.8, 40.8)
- added J2: Conn_01x06_Pin, Library:Pmod6, F.Cu at (111.4, 72.6)
- added J2: Conn_01x06_Pin, Library:Pmod6, F.Cu at (111.4, 50.1)
- added J2: Conn_01x06_Pin, Library:Pmod6, F.Cu at (111.4, 95.1)
- added J2: Conn_01x06_Pin, Library:Pmod6, F.Cu at (111.4, 27.5)
- added J3: Conn_01x03_Pin, Connector_PinHeader_2.54mm:PinHeader_1x03_P2.54mm_Vertical, F.Cu at (156.9, 94.8)
- added J3: Conn_01x03_Pin, Connector_PinHeader_2.54mm:PinHeader_1x03_P2.54mm_Vertical, F.Cu at (156.9, 49.8)
- added J3: Conn_01x03_Pin, Connector_PinHeader_2.54mm:PinHeader_1x03_P2.54mm_Vertical, F.Cu at (156.9, 27.3)
- added J3: Conn_01x03_Pin, Connector_PinHeader_2.54mm:PinHeader_1x03_P2.54mm_Vertical, F.Cu at (156.9, 72.3)
- added REF**: NPTH, NPTH, F.Cu at (186.0, 59.2)
- added REF**: NPTH, NPTH, F.Cu at (186.0, 60.7)
- added REF**: NPTH, NPTH, F.Cu at (186.0, 33.7)
- added REF**: NPTH, NPTH, F.Cu at (111.0, 35.2)
- added REF**: NPTH, NPTH, F.Cu at (150.0, 24.8)
- added REF**: NPTH, NPTH, F.Cu at (185.7, 115.5)
- added REF**: NPTH, NPTH, F.Cu at (150.0, 68.1)
- added REF**: NPTH, NPTH, F.Cu at (190.1, 25.0)
- added REF**: NPTH, NPTH, F.Cu at (111.3, 20.7)
- added REF**: NPTH, NPTH, F.Cu at (111.0, 99.7)
- added REF**: NPTH, NPTH, F.Cu at (111.0, 56.2)
- added REF**: NPTH, NPTH, F.Cu at (145.5, 90.6)
- added REF**: NPTH, NPTH, F.Cu at (111.0, 57.7)
- added REF**: NPTH, NPTH, F.Cu at (106.9, 25.0)
- added REF**: NPTH, NPTH, F.Cu at (111.0, 105.7)
- added REF**: NPTH, NPTH, F.Cu at (151.5, 24.8)
- added REF**: NPTH, NPTH, F.Cu at (111.0, 78.7)
- added REF**: NPTH, NPTH, F.Cu at (111.3, 117.2)
- added REF**: NPTH, NPTH, F.Cu at (150.0, 45.6)
- added REF**: NPTH, NPTH, F.Cu at (147.0, 69.8)
- added REF**: NPTH, NPTH, F.Cu at (185.7, 22.3)
- added REF**: NPTH, NPTH, F.Cu at (151.5, 47.3)
- added REF**: NPTH, NPTH, F.Cu at (186.0, 36.7)
- added REF**: NPTH, NPTH, F.Cu at (186.0, 56.2)
- added REF**: NPTH, NPTH, F.Cu at (148.5, 92.3)
- added REF**: NPTH, NPTH, F.Cu at (148.5, 45.6)
- added REF**: NPTH, NPTH, F.Cu at (147.0, 92.3)
- added REF**: NPTH, NPTH, F.Cu at (147.0, 24.8)
- added REF**: NPTH, NPTH, F.Cu at (145.5, 45.6)
- added REF**: NPTH, NPTH, F.Cu at (147.0, 45.6)
- added REF**: NPTH, NPTH, F.Cu at (150.0, 92.3)
- added REF**: NPTH, NPTH, F.Cu at (188.4, 112.9)
- added REF**: NPTH, NPTH, F.Cu at (106.9, 112.9)
- added REF**: NPTH, NPTH, F.Cu at (145.5, 92.3)
- added REF**: NPTH, NPTH, F.Cu at (186.0, 99.7)
- added REF**: NPTH, NPTH, F.Cu at (145.5, 113.1)
- added REF**: NPTH, NPTH, F.Cu at (111.3, 22.3)
- added REF**: NPTH, NPTH, F.Cu at (111.0, 81.7)
- added REF**: NPTH, NPTH, F.Cu at (186.0, 101.2)
- added REF**: NPTH, NPTH, F.Cu at (111.3, 115.5)
- added REF**: NPTH, NPTH, F.Cu at (151.5, 69.8)
- added REF**: NPTH, NPTH, F.Cu at (188.4, 25.0)
- added REF**: NPTH, NPTH, F.Cu at (111.0, 59.2)
- added REF**: NPTH, NPTH, F.Cu at (186.0, 105.7)
- added REF**: NPTH, NPTH, F.Cu at (148.5, 69.8)
- added REF**: NPTH, NPTH, F.Cu at (147.0, 90.6)
- added REF**: NPTH, NPTH, F.Cu at (147.0, 47.3)
- added REF**: NPTH, NPTH, F.Cu at (186.0, 78.7)
- added REF**: NPTH, NPTH, F.Cu at (150.0, 47.3)
- added REF**: NPTH, NPTH, F.Cu at (111.0, 54.7)
- added REF**: NPTH, NPTH, F.Cu at (186.0, 35.2)
- added REF**: NPTH, NPTH, F.Cu at (145.5, 69.8)
- added REF**: NPTH, NPTH, F.Cu at (111.0, 83.2)
- added REF**: NPTH, NPTH, F.Cu at (111.0, 104.2)
- added REF**: NPTH, NPTH, F.Cu at (151.5, 90.6)
- added REF**: NPTH, NPTH, F.Cu at (111.0, 80.2)
- added REF**: NPTH, NPTH, F.Cu at (111.0, 102.7)
- added REF**: NPTH, NPTH, F.Cu at (111.0, 60.7)
- added REF**: NPTH, NPTH, F.Cu at (186.0, 38.2)
- added REF**: NPTH, NPTH, F.Cu at (145.5, 24.8)
- added REF**: NPTH, NPTH, F.Cu at (111.0, 32.2)
- added REF**: NPTH, NPTH, F.Cu at (148.5, 90.6)
- added REF**: NPTH, NPTH, F.Cu at (186.0, 102.7)
- added REF**: NPTH, NPTH, F.Cu at (108.6, 112.9)
- added REF**: NPTH, NPTH, F.Cu at (186.0, 80.2)
- added REF**: NPTH, NPTH, F.Cu at (151.5, 92.3)
- added REF**: NPTH, NPTH, F.Cu at (150.0, 90.6)
- added REF**: NPTH, NPTH, F.Cu at (145.5, 68.1)
- added REF**: NPTH, NPTH, F.Cu at (186.0, 81.7)
- added REF**: NPTH, NPTH, F.Cu at (186.0, 32.2)
- added REF**: NPTH, NPTH, F.Cu at (148.5, 113.1)
- added REF**: NPTH, NPTH, F.Cu at (190.1, 112.9)
- added REF**: NPTH, NPTH, F.Cu at (145.5, 47.3)
- added REF**: NPTH, NPTH, F.Cu at (151.5, 113.1)
- added REF**: NPTH, NPTH, F.Cu at (185.7, 117.2)
- added REF**: NPTH, NPTH, F.Cu at (111.0, 38.2)
- added REF**: NPTH, NPTH, F.Cu at (111.0, 36.7)
- added REF**: NPTH, NPTH, F.Cu at (147.0, 68.1)
- added REF**: NPTH, NPTH, F.Cu at (108.6, 25.0)
- added REF**: NPTH, NPTH, F.Cu at (151.5, 68.1)
- added REF**: NPTH, NPTH, F.Cu at (186.0, 83.2)
- added REF**: NPTH, NPTH, F.Cu at (186.0, 104.2)
- added REF**: NPTH, NPTH, F.Cu at (151.5, 45.6)
- added REF**: NPTH, NPTH, F.Cu at (148.5, 68.1)
- added REF**: NPTH, NPTH, F.Cu at (111.0, 33.7)
- added REF**: NPTH, NPTH, F.Cu at (148.5, 47.3)
- added REF**: NPTH, NPTH, F.Cu at (150.0, 69.8)
- added REF**: NPTH, NPTH, F.Cu at (150.0, 113.1)
- added REF**: NPTH, NPTH, F.Cu at (111.0, 101.2)
- added REF**: NPTH, NPTH, F.Cu at (186.0, 57.7)
- added REF**: NPTH, NPTH, F.Cu at (147.0, 113.1)
- added REF**: NPTH, NPTH, F.Cu at (186.0, 54.7)
- added REF**: NPTH, NPTH, F.Cu at (111.0, 77.2)
- added REF**: NPTH, NPTH, F.Cu at (185.7, 20.7)
- added REF**: NPTH, NPTH, F.Cu at (148.5, 24.8)
- added REF**: NPTH, NPTH, F.Cu at (186.0, 77.2)
- added Reserve: TestPoint, TestPoint:TestPoint_Pad_D2.0mm, F.Cu at (135.1, 108.6)
- added Reserve: TestPoint, TestPoint:TestPoint_Pad_D2.0mm, F.Cu at (135.1, 41.0)
- added Reserve: TestPoint, TestPoint:TestPoint_Pad_D2.0mm, F.Cu at (135.1, 86.0)
- added Reserve: TestPoint, TestPoint:TestPoint_Pad_D2.0mm, F.Cu at (135.1, 63.5)
Other:
- board size 86.5 x 99.3 mm -> 84.5 x 97.9 mm

Commit message: 618
Parts:
- removed the D3 at (161.6, 110.7)
- removed the D3 at (161.6, 43.2)
- removed the D3 at (161.6, 88.2)
- removed the D3 at (161.6, 65.7)
- removed the G*** at (175.4, 74.5)
- removed the G*** at (175.4, 97.0)
- removed the G*** at (175.4, 52.0)
- removed the G*** at (175.4, 29.5)
- removed the IC1 at (127.5, 34.5)
- removed the IC1 at (127.5, 79.6)
- removed the IC1 at (127.5, 57.1)
- removed the IC1 at (127.5, 102.1)
- removed IC2 (x4): LM2940T-5.0, SamacSys_Parts:TO254P470X1016X2222-3P
- removed the J1 at (171.8, 63.3)
- removed the J1 at (171.8, 108.4)
- removed the J1 at (171.8, 85.9)
- removed the J1 at (171.8, 40.8)
- removed the REF** at (186.0, 59.2)
- removed the REF** at (186.0, 60.7)
- removed the REF** at (186.0, 33.7)
- removed the REF** at (111.0, 35.2)
- removed the REF** at (150.0, 24.8)
- removed the REF** at (150.0, 68.1)
- removed the REF** at (111.0, 99.7)
- removed the REF** at (111.0, 56.2)
- removed the REF** at (145.5, 90.6)
- removed the REF** at (111.0, 57.7)
- removed the REF** at (111.0, 105.7)
- removed the REF** at (151.5, 24.8)
- removed the REF** at (111.0, 78.7)
- removed the REF** at (150.0, 45.6)
- removed the REF** at (147.0, 69.8)
- removed the REF** at (151.5, 47.3)
- removed the REF** at (186.0, 36.7)
- removed the REF** at (186.0, 56.2)
- removed the REF** at (148.5, 92.3)
- removed the REF** at (148.5, 45.6)
- removed the REF** at (147.0, 92.3)
- removed the REF** at (147.0, 24.8)
- removed the REF** at (145.5, 45.6)
- removed the REF** at (147.0, 45.6)
- removed the REF** at (150.0, 92.3)
- removed the REF** at (145.5, 92.3)
- removed the REF** at (186.0, 99.7)
- removed the REF** at (145.5, 113.1)
- removed the REF** at (111.0, 81.7)
- removed the REF** at (186.0, 101.2)
- removed the REF** at (151.5, 69.8)
- removed the REF** at (111.0, 59.2)
- removed the REF** at (186.0, 105.7)
- removed the REF** at (148.5, 69.8)
- removed the REF** at (147.0, 90.6)
- removed the REF** at (147.0, 47.3)
- removed the REF** at (186.0, 78.7)
- removed the REF** at (150.0, 47.3)
- removed the REF** at (111.0, 54.7)
- removed the REF** at (186.0, 35.2)
- removed the REF** at (145.5, 69.8)
- removed the REF** at (111.0, 83.2)
- removed the REF** at (111.0, 104.2)
- removed the REF** at (151.5, 90.6)
- removed the REF** at (111.0, 80.2)
- removed the REF** at (111.0, 102.7)
- removed the REF** at (111.0, 60.7)
- removed the REF** at (186.0, 38.2)
- removed the REF** at (145.5, 24.8)
- removed the REF** at (111.0, 32.2)
- removed the REF** at (148.5, 90.6)
- removed the REF** at (186.0, 102.7)
- removed the REF** at (186.0, 80.2)
- removed the REF** at (151.5, 92.3)
- removed the REF** at (150.0, 90.6)
- removed the REF** at (145.5, 68.1)
- removed the REF** at (186.0, 81.7)
- removed the REF** at (186.0, 32.2)
- removed the REF** at (148.5, 113.1)
- removed the REF** at (145.5, 47.3)
- removed the REF** at (151.5, 113.1)
- removed the REF** at (111.0, 38.2)
- removed the REF** at (111.0, 36.7)
- removed the REF** at (147.0, 68.1)
- removed the REF** at (151.5, 68.1)
- removed the REF** at (186.0, 83.2)
- removed the REF** at (186.0, 104.2)
- removed the REF** at (151.5, 45.6)
- removed the REF** at (148.5, 68.1)
- removed the REF** at (111.0, 33.7)
- removed the REF** at (148.5, 47.3)
- removed the REF** at (150.0, 69.8)
- removed the REF** at (150.0, 113.1)
- removed the REF** at (111.0, 101.2)
- removed the REF** at (186.0, 57.7)
- removed the REF** at (147.0, 113.1)
- removed the REF** at (186.0, 54.7)
- removed the REF** at (111.0, 77.2)
- removed the REF** at (148.5, 24.8)
- removed the REF** at (186.0, 77.2)
- removed Reserve (x4): TestPoint, TestPoint:TestPoint_Pad_D2.0mm
- added C1: 0.1u, Capacitor_SMD:C_0603_1608Metric_Pad1.08x0.95mm_HandSolder, F.Cu at (183.0, 56.7)
- added C1: 0.1u, Capacitor_SMD:C_0603_1608Metric_Pad1.08x0.95mm_HandSolder, F.Cu at (183.0, 101.7)
- added C1: 0.1u, Capacitor_SMD:C_0603_1608Metric_Pad1.08x0.95mm_HandSolder, F.Cu at (183.0, 34.2)
- added C1: 0.1u, Capacitor_SMD:C_0603_1608Metric_Pad1.08x0.95mm_HandSolder, F.Cu at (183.0, 79.2)
- added C2: 0.1u, Capacitor_SMD:C_0603_1608Metric_Pad1.08x0.95mm_HandSolder, F.Cu at (171.0, 28.1)
- added C2: 0.1u, Capacitor_SMD:C_0603_1608Metric_Pad1.08x0.95mm_HandSolder, F.Cu at (171.0, 50.7)
- added C2: 0.1u, Capacitor_SMD:C_0603_1608Metric_Pad1.08x0.95mm_HandSolder, F.Cu at (171.0, 73.2)
- added C2: 0.1u, Capacitor_SMD:C_0603_1608Metric_Pad1.08x0.95mm_HandSolder, F.Cu at (171.0, 95.7)
- added D3: SS2040FL, SamacSys_Parts:SODFL3618X108N, F.Cu at (161.6, 65.2)
- added D3: SS2040FL, SamacSys_Parts:SODFL3618X108N, F.Cu at (161.6, 110.2)
- added D3: SS2040FL, SamacSys_Parts:SODFL3618X108N, F.Cu at (161.6, 87.7)
- added D3: SS2040FL, SamacSys_Parts:SODFL3618X108N, F.Cu at (161.6, 42.7)
- added G***: LOGO, MyLibrary:logo_kamo_ss, B.Cu at (128.0, 56.5)
- added G***: LOGO, MyLibrary:logo_kamo_ss, B.Cu at (128.0, 101.6)
- added G***: LOGO, MyLibrary:logo_kamo_ss, B.Cu at (128.0, 79.1)
- added G***: LOGO, MyLibrary:logo_kamo_ss, B.Cu at (128.0, 34.0)
- added IC1: TBD62064APG, SamacSys_Parts:DIP762W60P254L1975H445Q16N, F.Cu at (127.5, 79.3)
- added IC1: TBD62064APG, SamacSys_Parts:DIP762W60P254L1975H445Q16N, F.Cu at (127.5, 56.8)
- added IC1: TBD62064APG, SamacSys_Parts:DIP762W60P254L1975H445Q16N, F.Cu at (127.5, 34.3)
- added IC1: TBD62064APG, SamacSys_Parts:DIP762W60P254L1975H445Q16N, F.Cu at (127.5, 101.8)
- added J1: Barrel_Jack_Switch, Connector_BarrelJack:BarrelJack_Horizontal, F.Cu at (172.1, 108.1)
- added J1: Barrel_Jack_Switch, Connector_BarrelJack:BarrelJack_Horizontal, F.Cu at (172.1, 85.6)
- added J1: Barrel_Jack_Switch, Connector_BarrelJack:BarrelJack_Horizontal, F.Cu at (172.1, 63.0)
- added J1: Barrel_Jack_Switch, Connector_BarrelJack:BarrelJack_Horizontal, F.Cu at (172.1, 40.5)
- added REF**: NPTH, NPTH, F.Cu at (186.1, 58.4)
- added REF**: NPTH, NPTH, F.Cu at (147.0, 90.8)
- added REF**: NPTH, NPTH, F.Cu at (151.5, 92.2)
- added REF**: NPTH, NPTH, F.Cu at (186.1, 102.0)
- added REF**: NPTH, NPTH, F.Cu at (145.5, 113.3)
- added REF**: NPTH, NPTH, F.Cu at (186.1, 57.0)
- added REF**: NPTH, NPTH, F.Cu at (110.9, 82.3)
- added REF**: NPTH, NPTH, F.Cu at (186.1, 104.8)
- added REF**: NPTH, NPTH, F.Cu at (186.1, 37.3)
- added REF**: NPTH, NPTH, F.Cu at (110.9, 59.8)
- added REF**: NPTH, NPTH, F.Cu at (186.1, 33.1)
- added REF**: NPTH, NPTH, F.Cu at (186.1, 100.6)
- added REF**: NPTH, NPTH, F.Cu at (145.5, 90.8)
- added REF**: NPTH, NPTH, F.Cu at (110.9, 80.9)
- added REF**: NPTH, NPTH, F.Cu at (148.5, 90.8)
- added REF**: NPTH, NPTH, F.Cu at (186.1, 82.3)
- added REF**: NPTH, NPTH, F.Cu at (110.9, 100.6)
- added REF**: NPTH, NPTH, F.Cu at (148.5, 92.2)
- added REF**: NPTH, NPTH, F.Cu at (145.5, 69.6)
- added REF**: NPTH, NPTH, F.Cu at (145.5, 68.2)
- added REF**: NPTH, NPTH, F.Cu at (147.0, 69.6)
- added REF**: NPTH, NPTH, F.Cu at (110.9, 79.5)
- added REF**: NPTH, NPTH, F.Cu at (150.0, 113.3)
- added REF**: NPTH, NPTH, F.Cu at (148.5, 47.1)
- added REF**: NPTH, NPTH, F.Cu at (147.0, 47.1)
- added REF**: NPTH, NPTH, F.Cu at (145.5, 92.2)
- added REF**: NPTH, NPTH, F.Cu at (148.5, 45.7)
- added REF**: NPTH, NPTH, F.Cu at (110.9, 58.4)
- added REF**: NPTH, NPTH, F.Cu at (150.0, 69.6)
- added REF**: NPTH, NPTH, F.Cu at (186.1, 103.4)
- added REF**: NPTH, NPTH, F.Cu at (150.0, 47.1)
- added REF**: NPTH, NPTH, F.Cu at (186.1, 59.8)
- added REF**: NPTH, NPTH, F.Cu at (145.5, 24.6)
- added REF**: NPTH, NPTH, F.Cu at (147.0, 24.6)
- added REF**: NPTH, NPTH, F.Cu at (145.5, 47.1)
- added REF**: NPTH, NPTH, F.Cu at (150.0, 45.7)
- added REF**: NPTH, NPTH, F.Cu at (110.9, 33.1)
- added REF**: NPTH, NPTH, F.Cu at (150.0, 92.2)
- added REF**: NPTH, NPTH, F.Cu at (150.0, 24.6)
- added REF**: NPTH, NPTH, F.Cu at (150.0, 68.2)
- added REF**: NPTH, NPTH, F.Cu at (147.0, 68.2)
- added REF**: NPTH, NPTH, F.Cu at (148.5, 68.2)
- added REF**: NPTH, NPTH, F.Cu at (150.0, 90.8)
- added REF**: NPTH, NPTH, F.Cu at (110.9, 78.1)
- added REF**: NPTH, NPTH, F.Cu at (147.0, 45.7)
- added REF**: NPTH, NPTH, F.Cu at (151.5, 24.6)
- added REF**: NPTH, NPTH, F.Cu at (186.1, 80.9)
- added REF**: NPTH, NPTH, F.Cu at (151.5, 69.6)
- added REF**: NPTH, NPTH, F.Cu at (151.5, 90.8)
- added REF**: NPTH, NPTH, F.Cu at (151.5, 45.7)
- added REF**: NPTH, NPTH, F.Cu at (186.1, 35.9)
- added REF**: NPTH, NPTH, F.Cu at (110.9, 103.4)
- added REF**: NPTH, NPTH, F.Cu at (147.0, 113.3)
- added REF**: NPTH, NPTH, F.Cu at (110.9, 55.6)
- added REF**: NPTH, NPTH, F.Cu at (148.5, 69.6)
- added REF**: NPTH, NPTH, F.Cu at (147.0, 92.2)
- added REF**: NPTH, NPTH, F.Cu at (145.5, 45.7)
- added REF**: NPTH, NPTH, F.Cu at (110.9, 37.3)
- added REF**: NPTH, NPTH, F.Cu at (148.5, 24.6)
- added REF**: NPTH, NPTH, F.Cu at (110.9, 35.9)
- added REF**: NPTH, NPTH, F.Cu at (186.1, 55.6)
- added REF**: NPTH, NPTH, F.Cu at (186.1, 34.5)
- added REF**: NPTH, NPTH, F.Cu at (186.1, 78.1)
- added REF**: NPTH, NPTH, F.Cu at (110.9, 34.5)
- added REF**: NPTH, NPTH, F.Cu at (151.5, 47.1)
- added REF**: NPTH, NPTH, F.Cu at (110.9, 57.0)
- added REF**: NPTH, NPTH, F.Cu at (110.9, 102.0)
- added REF**: NPTH, NPTH, F.Cu at (151.5, 68.2)
- added REF**: NPTH, NPTH, F.Cu at (186.1, 79.5)
- added REF**: NPTH, NPTH, F.Cu at (110.9, 104.8)
- added REF**: NPTH, NPTH, F.Cu at (148.5, 113.3)
- added REF**: NPTH, NPTH, F.Cu at (151.5, 113.3)
- added U1: AMS1117-3.3, Package_TO_SOT_SMD:SOT-223-3_TabPin2, F.Cu at (177.3, 29.8)
- added U1: AMS1117-3.3, Package_TO_SOT_SMD:SOT-223-3_TabPin2, F.Cu at (177.3, 97.4)
- added U1: AMS1117-3.3, Package_TO_SOT_SMD:SOT-223-3_TabPin2, F.Cu at (177.3, 74.8)
- added U1: AMS1117-3.3, Package_TO_SOT_SMD:SOT-223-3_TabPin2, F.Cu at (177.3, 52.3)
Connections:
- D1 pad 2: Board_3-Net-(IC1-O2) -> Board_3-Net-(IC1-O4)
- D1 pad 2: Board_2-Net-(IC1-O2) -> Board_2-Net-(IC1-O4)
- D1 pad 2: Board_0-Net-(IC1-O2) -> Board_0-Net-(IC1-O4)
- D1 pad 2: Board_1-Net-(IC1-O2) -> Board_1-Net-(IC1-O4)
- J2 pad : (no net) -> Board_1-vcc
- J2 pad : (no net) -> Board_0-vcc
- J2 pad : (no net) -> Board_2-vcc
- J2 pad : (no net) -> Board_3-vcc
- J3 pad : (no net) -> Board_1-/ExVcc
- J3 pad : (no net) -> Board_2-/ExVcc
- J3 pad : (no net) -> Board_3-/ExVcc
- J3 pad : (no net) -> Board_0-/ExVcc
Routing:
- net Board_3-VCC: track 62.2 -> 0.00 mm
- net Board_0-VCC: track 62.2 -> 0.00 mm
- net Board_1-VCC: track 62.2 -> 0.00 mm
- net Board_2-VCC: track 62.2 -> 0.00 mm
- net Board_2-vcc: track 0.00 -> 61.7 mm
- net Board_1-vcc: track 0.00 -> 61.7 mm
- net Board_0-vcc: track 0.00 -> 61.7 mm
- net Board_3-vcc: track 0.00 -> 61.7 mm
- net Board_3-Net-(U1-VI): track 0.00 -> 32.8 mm
- net Board_2-Net-(U1-VI): track 0.00 -> 32.8 mm
- net Board_0-Net-(U1-VI): track 0.00 -> 32.8 mm
- net Board_1-Net-(U1-VI): track 0.00 -> 32.8 mm
- net Board_3-Net-(IC2-IN): track 22.4 -> 0.00 mm
- net Board_2-Net-(IC2-IN): track 22.4 -> 0.00 mm
- net Board_0-Net-(IC2-IN): track 22.4 -> 0.00 mm
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Other:
- outline, holes or cut-outs redrawn
- board text added: "Pmod_Color_LED Ver. 0.2"
- board text added: "[AZ1117 CH-3.3]"
- board text removed: "Pmod_Color_LED Ver. 0.1"
- board text removed: "[LM2940T -3.3]"
