File: Pmod_7LED_8digit/Pmod_7LED_8digit.kicad_pcb (KiCad board)
At the start: 2 copper layers, 15 parts, among them J1 Pmod_Header, U1 74HC595, U2 74HC595

Commit message: 0811
Parts:
- added G***: LOGO, MyLibrary:kamo20, B.Cu at (114.0, 74.2)
- moved J1 11.4 mm to (56.6, 68.3)
Routing:
- net Net-(DS1-ANODE_E_DIG_1234): track 68.4 -> 76.3 mm
- net Net-(DS1-ANODE_D_DIG_1234): track 75.0 -> 82.7 mm, vias 1 -> 3
- net Net-(DS2-COMMON_CATHODE_DIG_4): track 31.1 -> 36.5 mm
- net Net-(DS1-COMMON_CATHODE_DIG_4): track 78.4 -> 80.6 mm
- net Net-(DS1-COMMON_CATHODE_DIG_3): track 73.9 -> 75.7 mm
- net Net-(DS2-COMMON_CATHODE_DIG_2): track 21.6 -> 19.8 mm
- net Net-(J1-Pin_2): track 18.6 -> 16.9 mm
- net Net-(DS1-COMMON_CATHODE_DIG_2): track 70.4 -> 72.0 mm
- net Net-(J1-Pin_1): track 47.9 -> 46.4 mm
- net Net-(DS1-ANODE_G_DIG_1234): track 76.7 -> 75.6 mm
- net Net-(DS1-ANODE_C_DIG_1234): track 76.4 -> 77.2 mm
- net Net-(J1-Pin_3): track 14.8 -> 14.2 mm
- net GND: vias 0 -> 14
- added copper zone on B.Cu, net GND
- added copper zone on F.Cu, net GND
Other:
- board outline added: 99.6 x 20.3 mm
- board text added: "Pmod_8Digits_7SegLED"

Commit message: 0811
Changed lines of the file:
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@@
         (effects (font (size 1.27 1.27) (thickness 0.254)))
     )
-    (fp_line (start -2.005 -18.925) (end -2.005 0)
-      (stroke (width 0.2) (type solid)) (layer "F.SilkS"))
+    (fp_circle (center 0 -2.2) (end 0.3 -2.2)
+      (stroke (width 0.1) (type solid)) (fill solid) (layer "F.SilkS"))
     (fp_line (start -2.255 -19.175) (end 17.495 -19.175)
       (stroke (width 0.05) (type solid)) (layer "F.CrtYd"))
@@
         (effects (font (size 1.27 1.27) (thickness 0.254)))
     )
-    (fp_line (start -2.005 -18.925) (end -2.005 0)
-      (stroke (width 0.2) (type solid)) (layer "F.SilkS"))
+    (fp_circle (center 0 -2.2) (end 0.360555 -2.2)
+      (stroke (width 0.1) (type solid)) (fill solid) (layer "F.SilkS"))
     (fp_line (start -2.255 -19.175) (end 17.495 -19.175)
       (stroke (width 0.05) (type solid)) (layer "F.CrtYd"))

Commit message: 0830
Parts:
- moved G*** 1.14 mm to (115.2, 74.2)
Routing:
- net VCC: track 37.5 -> 39.7 mm
- net Net-(DS1-ANODE_D_DIG_1234): track 82.7 -> 81.6 mm
- net GND: vias 14 -> 15
Other:
- board text added: "Pmod_8Digits_7SegLED Ver0.2"
- board text removed: "Pmod_8Digits_7SegLED"
