File: Pmod_Matrix256/Pmod_Matrix256.kicad_pcb (KiCad board)
At the start: 2 copper layers, 92.6 x 42.2 mm, 22 parts, among them J1 Pmod_Header, U1 OSLB56317-ARA, U2 74AHC595, U3 74AHC595, U4 74AHC595, U5 74AHC595

Commit message: 811
Parts:
- moved J1 15.9 mm to (100.6, 119.4)
Routing:
- net VCC: track 135.3 -> 149.2 mm
- net /SRCLK: track 86.7 -> 87.8 mm
- net /#SRCLR: track 98.6 -> 97.7 mm
- net /RCLK: track 75.0 -> 75.6 mm
- net /SER1: track 18.6 -> 19.2 mm
- net GND: vias 8 -> 11
Other:
- board text added: "#EN"
- board text added: "#SRCLR"
- board text added: "G"
- board text added: "Pmod_MatrixLED256 Ver 0.1"
- board text added: "RCLK"
- board text added: "SER"
- board text added: "SRCLK"
- board text added: "[OSLB56317-ARA]"
- board text removed: "SUGAmod_MatrixLED256 Ver 0.1"

Commit message: 0812
Parts:
- added G***: LOGO, MyLibrary:kamo20, F.Cu at (104.6, 103.9)

Commit message: 0830
Other:
- board text added: "Anode"
- board text added: "COL1"
- board text added: "COL10"
- board text added: "COL11"
- board text added: "COL12"
- board text added: "COL13"
- board text added: "COL14"
- board text added: "COL15"
- board text added: "COL16"
- board text added: "COL2"
- board text added: "COL3"
- board text added: "COL4"
- board text added: "COL5"
- board text added: "COL6"
- board text added: "COL7"
- board text added: "COL8"
- board text added: "COL9"
- board text added: "Cathode Common"
- board text added: "Pmod_MatrixLED256 Ver 0.2"
- board text added: "ROW1"
- board text added: "ROW10"
- board text added: "ROW11"
- board text added: "ROW12"
- board text added: "ROW13"
- board text added: "ROW14"
- board text added: "ROW15"
- board text added: "ROW16"
- board text added: "ROW2"
- board text added: "ROW3"
- board text added: "ROW4"
- board text added: "ROW5"
- board text added: "ROW6"
- board text added: "ROW7"
- board text added: "ROW8"
- board text added: "ROW9"
- board text added: "[74HC595]"
- board text removed: "Pmod_MatrixLED256 Ver 0.1"
