File: Pmod_7Seg/Pmod_7Seg/Pmod_7Seg.kicad_pcb (KiCad board)
At the start: 2 copper layers, 68.5 x 42.4 mm, 14 parts, among them IC1 TBD62783APG, IC2 TBD62003APG, IC3 OSL60362-LR, J1 Conn_02x06_Counter_Clockwise, J2 Conn_02x06_Counter_Clockwise

Commit message: 0830
Parts:
- moved J2 11.3 mm to (112.5, 88.9)
- moved J1 11.2 mm to (112.5, 66.0)
Other:
- board text added: "Pmod_6gidit_7SegLED Ver 0.2"
- board text removed: "Pmod_6gidit_7SegLED Ver 0.1"
