File: Pmod_US_Speaker/Pmod_US_Speaker.kicad_pcb (KiCad board)
At the start: 2 copper layers, 99.3 x 20.3 mm, 18 parts, among them IC1 IR4427STRPBF, IC2 IR4427STRPBF, IC3 IR4427STRPBF, J1 Pmod_Header, J2 Barrel_Jack_Switch, J3 Conn_01x03, U1 CUSA-T80-18-2400-TH, U2 CUSA-T80-18-2400-TH, U3 CUSA-T80-18-2400-TH

Commit message: 1030
Parts:
- moved C2 0.20 mm to (166.4, 94.9)
Routing:
- net GND: track 9.33 -> 2.56 mm, vias 0 -> 4
Other:
- board text added: "G"
- board text added: "V"

Commit message: 1031
Parts:
- added G***: LOGO, MyLibrary:kamo20, B.Cu at (177.8, 101.0)
