File: Pmod_ADC/Pmod_ADC.kicad_pcb (KiCad board)
At the start: 2 copper layers, 99.6 x 20.3 mm, 29 parts, among them J1 Pmod_Header, J2 AudioJack3, J3 Screw_Terminal_01x03, J4 Conn_01x08, J5 Conn_02x02_Counter_Clockwise, U1 MCP3008, U3 MCP6492T

Commit message: 1201
Parts:
- removed J3: Screw_Terminal_01x03, TerminalBlock:TerminalBlock_bornier-3_P5.08mm
- U3: value MCP6492T -> [MCP6492T]
- moved TP1 79.3 mm to (217.0, 84.6)
- moved TP2 78.9 mm to (217.0, 89.2)
- moved C4 57.7 mm to (207.0, 91.2), turned to 180 degrees
- moved C3 57.3 mm to (202.2, 99.6), turned to 90 degrees
- moved R4 54.1 mm to (204.2, 99.6), turned to -90 degrees
- moved RV1 49.1 mm to (188.7, 94.0), turned to 180 degrees
- moved R9 47.9 mm to (199.9, 99.6), turned to 90 degrees
- moved R10 46.9 mm to (202.7, 95.2), turned to 180 degrees
- moved C2 44.8 mm to (185.0, 99.9), turned to -90 degrees
- moved R8 39.3 mm to (193.3, 91.4)
- moved R1 37.2 mm to (181.8, 96.8)
- moved J5 33.7 mm to (196.9, 97.5), turned to -90 degrees
- moved R2 32.9 mm to (178.3, 96.8)
- moved C1 30.2 mm to (160.3, 97.3), turned to 180 degrees
- moved JP1 29.0 mm to (181.9, 94.0), turned to 180 degrees
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Connections:
- net Net-(J4-Pin_8) renamed /CH0
- U1 pad 10: Net-(J1-Pin_1) -> Net-(J1-Pin_4)
- U1 pad 11: Net-(J1-Pin_2) -> Net-(J1-Pin_3)
- U1 pad 12: Net-(J1-Pin_3) -> Net-(J1-Pin_2)
- U1 pad 13: Net-(J1-Pin_4) -> Net-(J1-Pin_1)
Routing:
- net VCC: track 0.00 -> 78.9 mm
- net Net-(J1-Pin_1): track 0.00 -> 33.7 mm
- net Net-(J1-Pin_2): track 0.00 -> 29.7 mm
- net /CH0: track 0.00 -> 26.5 mm
- net Net-(J1-Pin_3): track 0.00 -> 25.6 mm
- net Net-(U3-V_INB+): track 0.00 -> 23.0 mm, vias 0 -> 2
- net Net-(J1-Pin_4): track 0.00 -> 21.6 mm
- net Net-(JP1-B): track 0.00 -> 17.1 mm
- net Net-(J4-Pin_1): track 0.00 -> 12.6 mm
- net Net-(C7-Pad2): track 0.00 -> 12.3 mm
- net Net-(U3-V_INA-): track 0.00 -> 12.0 mm
- net Net-(J4-Pin_2): track 0.00 -> 10.6 mm
- net Net-(J4-Pin_7): track 0.00 -> 8.94 mm
- net Net-(J5-Pin_1): track 0.00 -> 7.94 mm, vias 0 -> 1
- net Net-(J4-Pin_3): track 0.00 -> 7.28 mm
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- added copper zone on B.Cu, net GND
- added copper zone on F.Cu, net GND
Other:
- board size 99.6 x 20.3 mm -> 76.5 x 20.3 mm
- board text added: "#CS/SHDN"
- board text added: "<- Input from Phone Jack"
- board text added: "CH1"
- board text added: "CH2"
- board text added: "CH3"
- board text added: "CH4"
- board text added: "CH5"
- board text added: "CH6"
- board text added: "CH7"
- board text added: "CH8"
- board text added: "CLK"
- board text added: "Din"
- board text added: "Dout"
- board text added: "GND"
- board text added: "Input from Test Point ->"
- board text added: "NC"
- board text added: "Pmod_ADC Ver 0.1"
- board text added: "VCC"
- board text added: "[MCP3008/3208]"

Commit message: 1201
Parts:
- renumbered TP2 to GND
Changed lines of the file:
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@@
     (property "ki_keywords" "test point tp")
     (attr exclude_from_pos_files)
-    (fp_text reference "TP2" (at 0 2.032) (layer "F.SilkS")
+    (fp_text reference "GND" (at 0 2.032) (layer "F.SilkS")
         (effects (font (size 1 1) (thickness 0.15)))
     )
@@
     (fp_arc (start -1.286611 0.626746) (mid -1.431146 -0.000698) (end -1.286 -0.628)
       (stroke (width 0.12) (type solid)) (layer "F.SilkS"))
-    (fp_arc (start -0.627362 -1.285823) (mid -0.000201 -1.430704) (end 0.627 -1.286)
+    (fp_arc (start -0.627362 -1.285823) (mid -0.000201 -1.430703) (end 0.627 -1.286)
       (stroke (width 0.12) (type solid)) (layer "F.SilkS"))
     (fp_arc (start 0.02428 1.43094) (mid -0.310437 1.397071) (end -0.628 1.286)

Commit message: 1202
Parts:
- added G***: LOGO, MyLibrary:logo_kamo_ss, B.Cu at (209.3, 88.4)
Other:
- board text added: "#CS"
- board text added: "CH0"
- board text added: "G"
- board text added: "Ref"

Commit message: 0104
Parts:
- U3: value [MCP6492T] -> MCP6492T
- moved R4 12.0 mm to (211.8, 90.3), turned to 180 degrees
- moved C3 10.7 mm to (207.5, 90.3), turned to 180 degrees
- moved R5 10.5 mm to (203.9, 99.1), turned to -90 degrees
- moved C4 9.44 mm to (201.9, 99.1), turned to 90 degrees
- moved R10 0.69 mm to (202.3, 95.8)
- moved R9 0.46 mm to (199.9, 99.1)
- renumbered GND to TP2
Connections:
- J2 pad S: Net-(J2-PadS) -> GND
- J2 pad T: GND -> Net-(J2-PadT)
- R4 pad 1: Net-(J2-PadR) -> Net-(J2-PadT)
- R5 pad 1: Net-(J2-PadS) -> Net-(J2-PadR)
Routing:
- net Net-(J2-PadS): track 6.53 -> 0.00 mm
- net Net-(J2-PadT): track 0.00 -> 3.96 mm
- net Net-(U3-V_INA-): track 12.0 -> 12.8 mm
- net Net-(J2-PadR): track 2.63 -> 3.18 mm
