File: Pmod_ADC/Pmod_ADC.kicad_sch (KiCad schematic)
At the start: 11 parts, among them J1 Pmod_Header, J2 AudioJack3, J3 Screw_Terminal_01x03, J4 Conn_01x08, U1 MCP3008

Commit message: 1010
Parts:
- added U2: MCP6022, symbol Amplifier_Operational:MCP6022
Changed lines of the file:
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@@
     (stroke (width 0) (type default))
+  )
+  (symbol (lib_id "Amplifier_Operational:MCP6022") (at 173.355 131.445 0) (unit 3)
+    (in_bom yes) (on_board yes) (dnp no) (fields_autoplaced)
+    (property "Reference" "U2" (at 171.45 131.445 0)
+      (effects (font (size 1.27 1.27)) (justify left) hide)
+    )
+    (property "Value" "MCP6022" (at 172.085 132.715 0)
+      (effects (font (size 1.27 1.27)) (justify left) hide)
+    )
+    (property "Footprint" "" (at 173.355 131.445 0)
+      (effects (font (size 1.27 1.27)) hide)
+    )
+    (property "Datasheet" "http://ww1.microchip.com/downloads/en/devicedoc/20001685e.pdf" (at 173.355 131.445 0)
+      (effects (font (size 1.27 1.27)) hide)
+    )
+    (pin "1")
+    (pin "2")
+    (pin "3")
+    (pin "5")
+    (pin "6")
+    (pin "7")
+    (pin "4")
+    (pin "8")
+    (instances
+      (project "Pmod_ADC"
+        (path "/05ea207d-0e3d-4f58-8017-6fcac7fa1a7d"
+          (reference "U2") (unit 3)
+        )
+      )
+    )
   )
   (symbol (lib_id "power:GND") (at 129.54 102.235 0) (unit 1)
@@
     )
   )
+  (symbol (lib_id "Amplifier_Operational:MCP6022") (at 173.355 131.445 0) (unit 1)
+    (in_bom yes) (on_board yes) (dnp no)
+    (property "Reference" "U2" (at 174.625 123.825 0)
+      (effects (font (size 1.27 1.27)))
+    )
+    (property "Value" "MCP6022" (at 177.165 125.73 0)
+      (effects (font (size 1.27 1.27)))
+    )
+    (property "Footprint" "" (at 173.355 131.445 0)
+      (effects (font (size 1.27 1.27)) hide)
+    )
+    (property "Datasheet" "http://ww1.microchip.com/downloads/en/devicedoc/20001685e.pdf" (at 173.355 131.445 0)
+      (effects (font (size 1.27 1.27)) hide)
+    )
+    (pin "1")
+    (pin "2")
+    (pin "3")
+    (pin "5")
+    (pin "6")
+    (pin "7")
+    (pin "4")
+    (pin "8")
+    (instances
+      (project "Pmod_ADC"
+        (path "/05ea207d-0e3d-4f58-8017-6fcac7fa1a7d"
+          (reference "U2") (unit 1)
+        )
+      )
+    )
+  )
   (symbol (lib_id "Connector:Screw_Terminal_01x03") (at 210.185 79.375 0) (unit 1)
     (in_bom yes) (on_board yes) (dnp no)
@@
         )
       )
+    )
+  )
+  (symbol (lib_id "Amplifier_Operational:MCP6022") (at 173.355 149.86 0) (unit 2)
+    (in_bom yes) (on_board yes) (dnp no)
+    (property "Reference" "U2" (at 174.625 142.875 0)
+      (effects (font (size 1.27 1.27)))
+    )
+    (property "Value" "MCP6022" (at 177.165 144.78 0)
+      (effects (font (size 1.27 1.27)))
+    )
+    (property "Footprint" "" (at 173.355 149.86 0)
+      (effects (font (size 1.27 1.27)) hide)
+    )
+    (property "Datasheet" "http://ww1.microchip.com/downloads/en/devicedoc/20001685e.pdf" (at 173.355 149.86 0)
+      (effects (font (size 1.27 1.27)) hide)
+    )
+    (pin "1")
+    (pin "2")
+    (pin "3")
+    (pin "5")
+    (pin "6")
+    (pin "7")
+    (pin "4")
+    (pin "8")
+    (instances
+      (project "Pmod_ADC"
+        (path "/05ea207d-0e3d-4f58-8017-6fcac7fa1a7d"
+          (reference "U2") (unit 2)
+        )
+      )

Commit message: 1129
Parts:
- removed R3: R_Variable, symbol Device:R_Variable
- removed U2: MCP6022, symbol Amplifier_Operational:MCP6022
- added C3, C4, C5, C7: 1u, Capacitor_SMD:C_0603_1608Metric_Pad1.08x0.95mm_HandSolder, symbol Device:C
- added C6: 0.1u, Capacitor_SMD:C_0603_1608Metric_Pad1.08x0.95mm_HandSolder, symbol Device:C
- added J5: Conn_02x02_Counter_Clockwise, Connector_PinHeader_2.54mm:PinHeader_2x02_P2.54mm_Vertical, symbol Connector_Generic:Conn_02x02_Counter_Clockwise
- added R10, R6, R7: 100k, Resistor_SMD:R_0603_1608Metric_Pad0.98x0.95mm_HandSolder, symbol Device:R
- added R11, R12: 220k1%, Resistor_SMD:R_0603_1608Metric_Pad0.98x0.95mm_HandSolder, symbol Device:R
- added R4, R5: 47k, Resistor_SMD:R_0603_1608Metric_Pad0.98x0.95mm_HandSolder, symbol Device:R
- added R8, R9: 22, Resistor_SMD:R_0603_1608Metric_Pad0.98x0.95mm_HandSolder, symbol Device:R
- added RV1: R_Potentiometer, samacsys:TSR3296W203R, symbol Device:R_Potentiometer
- added TP1, TP2: TestPoint, TestPoint:TestPoint_THTPad_1.5x1.5mm_Drill0.7mm, symbol Connector:TestPoint
- added U3: MCP6492T, Package_SO:SOIC-8_3.9x4.9mm_P1.27mm, symbol Library:MCP6492T
- R2: footprint (none) -> Resistor_SMD:R_0603_1608Metric_Pad0.98x0.95mm_HandSolder
- U1: footprint (none) -> Package_DIP:DIP-16_W7.62mm
Connections:
- net GND: now also J1.11 (Pin_11), J1.5 (Pin_5), C6.2, C7.1, R12.1, RV1.3, TP2.1, U3.4 (VSS)
- net VCC: now also J1.12 (Pin_12), J1.6 (Pin_6), J3.3 (Pin_3), C6.1, R11.1, RV1.1, U3.8 (VDD)
- net at J1.1 (Pin_1): now also U1.10 (~{CS}/SHDN)
- net at J1.2 (Pin_2): now also U1.11 (Din)
- net at J1.3 (Pin_3): now also U1.12 (Dout)
- net at J1.4 (Pin_4): now also U1.13 (CLK)
- net at JP1.2 (B), R1.1, R2.2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: now also RV1.2
- net at J4.8 (Pin_8), U1.1 (CH0): now also J5.3 (Pin_3), J5.4 (Pin_4); no longer J2.R
- net at J4.7 (Pin_7), U1.2 (CH1): now also J3.2 (Pin_2)
- net at J4.6 (Pin_6), U1.3 (CH2): no longer J3.2 (Pin_2)
- net at J2.S: now also R5.1
- new net: C5.1, TP1.1
- new net: C5.2, R6.1, U3.5 (V_INB+)
- new net: C4.1, R5.2
- new net: C7.2, R11.2, R12.2, R6.2, R7.2
- new net: C3.1, R4.2
- new net: C3.2, C4.2, R10.1, U3.2 (V_INA-)
- new net: R10.2, R9.2, U3.1 (VOUTA)
- new net: R7.1, U3.3 (V_INA+)
- new net: R8.2, U3.6 (V_INB-), U3.7 (V_OUTB)
- new net: J5.1 (Pin_1), R8.1
- new net: J2.R, R4.1
- new net: J5.2 (Pin_2), R9.1
Other:
- moved on the sheet: J1, J2, J4, JP1

Commit message: 1201
Parts:
- removed J3: Screw_Terminal_01x03, TerminalBlock:TerminalBlock_bornier-3_P5.08mm, symbol Connector:Screw_Terminal_01x03
Connections:
- net at J1.1 (Pin_1): now also U1.13 (CLK); no longer U1.10 (~{CS}/SHDN)
- net at J1.2 (Pin_2): now also U1.12 (Dout); no longer U1.11 (Din)
- net at J1.3 (Pin_3): now also U1.11 (Din); no longer U1.12 (Dout)
- net at J1.4 (Pin_4): now also U1.10 (~{CS}/SHDN); no longer U1.13 (CLK)
- net CH0: now reaches J4.8 (Pin_8), J5.3 (Pin_3), J5.4 (Pin_4), U1.1 (CH0)
- no-connect marks 0 -> 4
Other:
- moved on the sheet: R8

Commit message: 0104
Connections:
- net GND: now also J2.S; no longer J2.T
- net at R5.1: now also J2.R; no longer J2.S
- net at R4.1: now also J2.T; no longer J2.R
Other:
- moved on the sheet: J2
Changed lines of the file:
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@@
+    (stroke (width 0) (type default))
+  )
+  (wire (pts (xy 34.29 76.835) (xy 30.48 76.835))
     (stroke (width 0) (type default))
   )
@@
     (stroke (width 0) (type default))
   )
+  (wire (pts (xy 30.48 79.375) (xy 36.195 79.375))
+    (stroke (width 0) (type default))
+  )
   (wire (pts (xy 46.355 91.44) (xy 48.26 91.44))
     (stroke (width 0) (type default))
   )
-  (wire (pts (xy 34.29 77.47) (xy 34.29 69.215))
+  (wire (pts (xy 34.29 69.215) (xy 34.29 76.835))
     (stroke (width 0) (type default))
   )
@@
     (stroke (width 0) (type default))
   )
+  (wire (pts (xy 27.305 66.675) (xy 30.48 66.675))
+    (stroke (width 0) (type default))
+  )
   (wire (pts (xy 99.695 84.455) (xy 96.52 84.455))
     (stroke (width 0) (type default))
@@
     (stroke (width 0) (type default))
   )
+  (wire (pts (xy 30.48 66.675) (xy 30.48 74.295))
+    (stroke (width 0) (type default))
+  )
   (wire (pts (xy 121.285 128.27) (xy 121.285 132.08))
     (stroke (width 0) (type default))
@@
     (stroke (width 0) (type default))
   )
-  (wire (pts (xy 31.75 77.47) (xy 34.29 77.47))
-    (stroke (width 0) (type default))
-  )
   (wire (pts (xy 102.87 85.09) (xy 102.87 87.63))
     (stroke (width 0) (type default))
@@
     (stroke (width 0) (type default))
   )
-  (wire (pts (xy 31.75 80.01) (xy 36.195 80.01))
-    (stroke (width 0) (type default))
-  )
   (wire (pts (xy 36.195 117.475) (xy 38.1 117.475))
     (stroke (width 0) (type default))
@@
     (stroke (width 0) (type default))
   )
-  (wire (pts (xy 36.195 80.01) (xy 36.195 76.835))
+  (wire (pts (xy 36.195 76.835) (xy 36.195 79.375))
     (stroke (width 0) (type default))
   )
@@
         (path "/05ea207d-0e3d-4f58-8017-6fcac7fa1a7d"
           (reference "#PWR03") (unit 1)
+        )
+      )
+    )
+  )
+  (symbol (lib_id "power:GND") (at 27.305 66.675 0) (unit 1)
+    (in_bom yes) (on_board yes) (dnp no) (fields_autoplaced)
+    (property "Reference" "#PWR05" (at 27.305 73.025 0)
+      (effects (font (size 1.27 1.27)) hide)
+    )
+    (property "Value" "GND" (at 27.305 71.12 0)
+      (effects (font (size 1.27 1.27)))
+    )
+    (property "Footprint" "" (at 27.305 66.675 0)
+      (effects (font (size 1.27 1.27)) hide)
+    )
+    (property "Datasheet" "" (at 27.305 66.675 0)
+      (effects (font (size 1.27 1.27)) hide)
+    )
+    (pin "1")
+    (instances
+      (project "Pmod_ADC"
+        (path "/05ea207d-0e3d-4f58-8017-6fcac7fa1a7d"
+          (reference "#PWR05") (unit 1)
         )
       )
@@
     )
   )
-  (symbol (lib_id "power:GND") (at 31.75 82.55 0) (unit 1)
-    (in_bom yes) (on_board yes) (dnp no)
-    (property "Reference" "#PWR06" (at 31.75 88.9 0)
-      (effects (font (size 1.27 1.27)) hide)
-    )
-    (property "Value" "GND" (at 31.115 86.36 0)
-      (effects (font (size 1.27 1.27)))
-    )
-    (property "Footprint" "" (at 31.75 82.55 0)
-      (effects (font (size 1.27 1.27)) hide)
-    )
-    (property "Datasheet" "" (at 31.75 82.55 0)
-      (effects (font (size 1.27 1.27)) hide)
-    )
-    (pin "1")
-    (instances
-      (project "Pmod_ADC"
-        (path "/05ea207d-0e3d-4f58-8017-6fcac7fa1a7d"
-          (reference "#PWR06") (unit 1)
-        )
-      )
-    )
-  )
   (symbol (lib_id "power:VCC") (at 190.5 81.28 0) (unit 1)
     (in_bom yes) (on_board yes) (dnp no)
@@
     )
   )
-  (symbol (lib_id "Connector_Audio:AudioJack3") (at 26.67 80.01 0) (unit 1)
-    (in_bom yes) (on_board yes) (dnp no)
-    (property "Reference" "J2" (at 20.955 76.835 0)
+  (symbol (lib_id "Connector_Audio:AudioJack3") (at 25.4 76.835 0) (unit 1)
+    (in_bom yes) (on_board yes) (dnp no)
+    (property "Reference" "J2" (at 19.685 73.66 0)
       (effects (font (size 1.27 1.27)) (justify right))
     )
-    (property "Value" "AudioJack3" (at 26.035 74.295 0)
+    (property "Value" "AudioJack3" (at 24.765 71.12 0)
       (effects (font (size 1.27 1.27)) (justify right))
     )
-    (property "Footprint" "Connector_Audio:Jack_3.5mm_Switronic_ST-005-G_horizontal" (at 26.67 80.01 0)
-      (effects (font (size 1.27 1.27)) hide)
-    )
-    (property "Datasheet" "~" (at 26.67 80.01 0)
-      (effects (font (size 1.27 1.27)) hide)
-    )
+    (property "Footprint" "Connector_Audio:Jack_3.5mm_Switronic_ST-005-G_horizontal" (at 25.4 76.835 0)
+      (effects (font (size 1.27 1.27)) hide)
+    )
+    (property "Datasheet" "~" (at 25.4 76.835 0)
+      (effects (font (size 1.27 1.27)) hide)
+    )
