File: Pmod_CAN/Pmod_CAN.kicad_sch (KiCad schematic)
At the start: 8 parts, among them IC1 TJA1441AT, IC2 AE_XC9306-5V0, J1 B2B-XH-A_LF__SN_

Commit message: 0112
Parts:
- added D1: WS2812B, Resistor_THT:R_Axial_DIN0309_L9.0mm_D3.2mm_P2.54mm_Vertical, symbol LED:WS2812B
- added D2, D3: WS2812B, LED_SMD:LED_WS2812B_PLCC4_5.0x5.0mm_P3.2mm, symbol LED:WS2812B
- added J2: Pmod_Header, MyLibrary:Pmod, symbol MyLibrary:Pmod_Header
- added Q1: Q_NPN_BEC, Package_TO_SOT_SMD:SC-59_Handsoldering, symbol Device:Q_NPN_BEC
- added R5: 4.7k, Resistor_SMD:R_0603_1608Metric_Pad0.98x0.95mm_HandSolder, symbol Device:R
- added R6: 10k, Resistor_SMD:R_0603_1608Metric_Pad0.98x0.95mm_HandSolder, symbol Device:R
- IC1: footprint SOIC127P600X175-8N -> SamacSys_Parts:SOIC127P600X175-8N
- IC2: footprint (none) -> Library:AE-XC9306-5V0
- J1: footprint SHDR2W64P0X250_1X2_740X575X700P -> SamacSys_Parts:SHDR2W64P0X250_1X2_740X575X700P
- R1: footprint Resistor_THT:R_Axial_DIN0309_L9.0mm_D3.2mm_P12.70mm_Horizontal -> Resistor_THT:R_Axial_DIN0309_L9.0mm_D3.2mm_P2.54mm_Vertical
- R3: footprint (none) -> Resistor_SMD:R_0603_1608Metric_Pad0.98x0.95mm_HandSolder
Connections:
- net +3V3: now also J2.12 (Pin_12), J2.6 (Pin_6), R5.1
- net +5V: now also D1.1 (VDD), D2.1 (VDD), D3.1 (VDD), R6.2
- net GND: now also D1.3 (VSS), D2.3 (VSS), D3.3 (VSS), J2.11 (Pin_11), J2.5 (Pin_5)
- net at IC1.1 (TXD), R3.1: now also J2.3 (Pin_3)
- net at IC1.4 (RXD), R2.1: now also J2.2 (Pin_2)
- net at IC1.8 (S), R4.1: now also J2.1 (Pin_1)
- new net: Q1.1 (B), R5.2
- new net: D2.2 (DOUT), D3.4 (DIN)
- new net: D1.2 (DOUT), D2.4 (DIN)
- new net: D1.4 (DIN), Q1.3 (C), R6.1
- new net: J2.4 (Pin_4), Q1.2 (E)
- no-connect marks 3 -> 4
