File: Pmod_CAN/Pmod_CAN.kicad_pcb (KiCad board)
At the start: 2 copper layers, 32.3 x 20.6 mm, 15 parts, among them IC1 TJA1441AT, IC2 AE_XC9306-5V0, J1 B2B-XH-A_LF__SN_, J2 Pmod_Header, Q1 Q_NPN_BEC

Commit message: 0112
Parts:
- added G***: LOGO, logo:logo_kamo, B.Cu at (153.9, 97.7)
Other:
- board text added: "3V3"
- board text added: "5V"
- board text added: "GND"
- board text added: "Pmod_CAN Ver 0.1"
- board text added: "RXD"
- board text added: "RxD"
- board text added: "S"
- board text added: "TXD"
- board text added: "TxD"
- board text added: "WS2812B"

Commit message: 0117
Parts:
- moved J2 11.3 mm to (139.6, 91.8)
