File: Pmod_CAN/v2/Pmod_CAN.kicad_sch (KiCad schematic)
At the start: 20 parts, among them IC1 TJA1441AT, IC2 AE_XC9306-5V0, J1 B2B-XH-A_LF__SN_, J2 Pmod_Header, Q1 Q_NPN_BEC

Commit message: 0306
Connections:
- net at Q1.2 (E): now also J2.7 (Pin_7); no longer J2.10 (Pin_10)
- net at IC1.8 (S), R4.1: now also J2.8 (Pin_8); no longer J2.7 (Pin_7)
- net at IC1.4 (RXD), R2.1: now also J2.10 (Pin_10); no longer J2.8 (Pin_8)

Commit message: 0306
Parts:
- added J3: Conn_01x06, Connector_PinHeader_2.54mm:PinHeader_1x06_P2.54mm_Vertical, symbol Connector_Generic:Conn_01x06
- added J4: Conn_01x02, Connector_PinHeader_2.54mm:PinHeader_1x02_P2.54mm_Vertical, symbol Connector_Generic:Conn_01x02
Connections:
- net +3V3: now also J3.6 (Pin_6)
- net GND: now also J3.5 (Pin_5)
- net at D4.1, J1.2, L1.2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: now also J4.2 (Pin_2)
- net at D4.2, J1.1, L1.3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: now also J4.1 (Pin_1)
- net at IC1.1 (TXD), J2.9 (Pin_9), R3.1: now also J3.3 (Pin_3)
- net at J2.7 (Pin_7), Q1.2 (E): now also J3.1 (Pin_1)
- net at IC1.4 (RXD), J2.10 (Pin_10), R2.1: now also J3.4 (Pin_4)
- net at IC1.8 (S), J2.8 (Pin_8), R4.1: now also J3.2 (Pin_2)

Commit message: 0309
Changed lines of the file:
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@@
 		)
 		(property "Value" "AE_XC9306-5V0"
-			(at 143.51 141.605 90)
+			(at 140.97 141.605 90)
 			(effects
 				(font
@@
 			)
 		)
-		(pin "1"
+		(pin "6"
 		)
 		(pin "1"
@@
 		(pin "2"
 		)
-		(pin "2"
+		(pin "4"
 		)
 		(pin "3"
 		)
-		(pin "3"
+		(pin "5"
 		)
 		(instances
