File: Pmod_CAN/v2/Pmod_CAN.kicad_pcb (KiCad board)
At the start: 2 copper layers, 32.3 x 20.6 mm, 21 parts, among them IC1 TJA1441AT, IC2 AE_XC9306-5V0, J1 B2B-XH-A_LF__SN_, J2 Pmod_Header, Q1 Q_NPN_BEC

Commit message: 0304
Parts:
- moved L1 28.3 mm to (163.1, 103.6)
- moved D4 25.2 mm to (176.8, 87.2)
- moved C3 24.3 mm to (151.4, 102.6), turned to -90 degrees
- moved R7 23.3 mm to (163.1, 98.0)
- moved C2 23.2 mm to (154.9, 98.0), turned to 180 degrees
- moved R5 20.3 mm to (139.6, 86.9)
- moved R4 20.2 mm to (157.5, 100.1), turned to 180 degrees
- moved R2 19.9 mm to (154.9, 107.7)
- moved Q1 15.7 mm to (143.5, 86.5)
- moved R3 12.5 mm to (153.9, 100.1), turned to 0 degrees
- moved C1 11.0 mm to (151.4, 106.2), turned to 90 degrees
- moved R1 6.53 mm to (163.1, 96.5)
- moved J1 4.61 mm to (168.7, 99.2)
- moved IC2 4.06 mm to (146.3, 102.7)
- moved R6 1.85 mm to (143.8, 96.5)
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Routing:
- net Net-(IC1-RXD): track 31.9 -> 0.00 mm, vias 1 -> 0
- net +3V3: track 33.5 -> 2.54 mm, vias 1 -> 0
- net Net-(IC1-TXD): track 24.8 -> 0.00 mm, vias 1 -> 0
- net Net-(IC1-S): track 23.0 -> 0.00 mm, vias 1 -> 0
- net /+5V: track 39.1 -> 18.8 mm
- net Net-(D1-DIN): track 11.4 -> 0.00 mm
- net (no net): track 9.64 -> 0.00 mm, vias 1 -> 0
- net Net-(D4-Pad2): track 9.03 -> 0.00 mm
- net Net-(D4-Pad1): track 5.31 -> 0.00 mm
- net Net-(IC1-CANL): track 3.55 -> 0.00 mm
- net Net-(Q1-B): track 3.45 -> 0.00 mm
- net Net-(IC1-CANH): track 3.21 -> 0.00 mm
- net unconnected-(J2-Pin_4-Pad4): track 0.00 -> 0.81 mm
- net GND: vias 9 -> 0
Other:
- board size 32.3 x 20.6 mm -> 38.1 x 20.6 mm
- copper layers 2 -> 6

Commit message: 0305
Parts:
- moved D4 11.7 mm to (167.8, 94.6)
- moved C2 10.8 mm to (161.7, 106.4), turned to 0 degrees
- moved R1 8.25 mm to (161.7, 104.6)
- moved Q1 6.35 mm to (144.8, 92.7), turned to -90 degrees
- moved R5 5.50 mm to (144.7, 89.0)
- moved C3 4.69 mm to (155.3, 105.2), turned to 180 degrees
- moved R2 4.15 mm to (151.1, 106.0), turned to -90 degrees
- moved C1 3.99 mm to (155.3, 106.8), turned to 180 degrees
- moved IC1 3.01 mm to (154.2, 101.5)
- moved L1 2.88 mm to (161.2, 101.5)
- moved R3 2.50 mm to (153.3, 97.7)
- moved R4 2.44 mm to (157.9, 97.7), turned to 0 degrees
- moved J1 2.18 mm to (166.8, 100.2), turned to -90 degrees
- moved R6 1.78 mm to (145.5, 96.4)
- moved D1 1.46 mm to (149.5, 91.8)
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Routing:
- net unconnected-(J2-Pin_4-Pad4): track 0.81 -> 0.00 mm
- net /+5V: track 18.8 -> 18.2 mm
Other:
- board size 38.1 x 20.6 mm -> 37.3 x 20.6 mm

Commit message: 0306
Parts:
- moved G*** 17.1 mm to (156.6, 80.8)
- moved R5 6.95 mm to (142.5, 95.6), turned to 90 degrees
- moved R6 3.22 mm to (146.1, 93.2), turned to -90 degrees
- moved C2 2.47 mm to (160.6, 104.2), turned to 180 degrees
- moved Q1 2.16 mm to (143.4, 91.1), turned to 90 degrees
- moved R7 1.68 mm to (163.3, 97.8), turned to 90 degrees
- moved R1 1.66 mm to (163.3, 105.1), turned to 90 degrees
- moved R3 1.14 mm to (152.1, 97.7)
- moved D4 1.14 mm to (167.7, 93.5)
- moved C1 0.76 mm to (154.6, 106.8)
- moved C3 0.76 mm to (154.6, 105.2)
- moved R4 0.38 mm to (158.2, 97.7)
Connections:
- J2 pad 10: Net-(J2-Pin_10) -> Net-(IC1-RXD)
- J2 pad 7: Net-(IC1-S) -> Net-(J2-Pin_7)
- J2 pad 8: Net-(IC1-RXD) -> Net-(IC1-S)
- Q1 pad 2: Net-(J2-Pin_10) -> Net-(J2-Pin_7)
Routing:
- net +3V3: track 2.54 -> 30.7 mm, vias 0 -> 1
- net Net-(IC1-S): track 0.00 -> 23.7 mm, vias 0 -> 1
- net Net-(IC1-TXD): track 0.00 -> 20.5 mm, vias 0 -> 1
- net Net-(IC1-RXD): track 0.00 -> 17.9 mm
- net Net-(D4-Pad1): track 0.00 -> 16.7 mm, vias 0 -> 1
- net /+5V: track 18.2 -> 34.7 mm
- net Net-(C2-Pad1): track 0.00 -> 14.5 mm, vias 0 -> 2
- net Net-(D4-Pad2): track 0.00 -> 12.7 mm
- net Net-(J2-Pin_7): track 0.00 -> 11.0 mm
- net Net-(D1-DIN): track 0.00 -> 7.37 mm
- net Net-(IC1-CANL): track 0.00 -> 2.99 mm
- net Net-(IC1-CANH): track 0.00 -> 2.99 mm
- net Net-(Q1-B): track 0.00 -> 2.03 mm
- net GND: vias 0 -> 3
Other:
- board text removed: "RxD"
- board text removed: "TxD"

Commit message: 0306
Parts:
- added J3: Conn_01x06, Connector_PinHeader_2.54mm:PinHeader_1x06_P2.54mm_Vertical, F.Cu at (133.1, 91.8)
- added J4: Conn_01x02, Connector_PinHeader_2.54mm:PinHeader_1x02_P2.54mm_Vertical, F.Cu at (170.4, 100.2)
- moved G*** 16.9 mm to (154.3, 97.5)
Routing:
- net Net-(J4-Pin_2): track 16.7 -> 20.2 mm
- net Net-(J2-Pin_7): track 11.0 -> 14.5 mm
- net Net-(IC1-TXD): track 20.5 -> 23.9 mm
- net Net-(IC1-S): track 23.7 -> 27.2 mm
- net Net-(IC1-RXD): track 17.9 -> 21.4 mm
- net GND: track 2.54 -> 5.98 mm, vias 3 -> 5
- net +3V3: track 30.7 -> 34.2 mm
- net Net-(J4-Pin_1): track 12.7 -> 15.2 mm
Other:
- copper layers 6 -> 2

Commit message: 0309
Parts:
- moved R5 0.25 mm to (142.5, 95.4)
Routing:
- net /+5V: track 34.7 -> 57.3 mm, vias 0 -> 2
- net +3V3: track 34.2 -> 41.4 mm
- net Net-(IC1-S): track 27.2 -> 28.2 mm
- net Net-(IC1-RXD): vias 0 -> 1
- net GND: vias 5 -> 4
Other:
- board text added: "Pmod_CAN Ver 0.2"
- board text removed: "Pmod_CAN Ver 0.1"

Commit message: 0320
Parts:
- moved IC2 0.25 mm to (145.8, 102.4)
- moved J3 0.13 mm to (133.2, 91.8)
- moved J4 0.13 mm to (170.3, 100.2)
Routing:
- net GND: vias 4 -> 7
Changed lines of the file:
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@@
 	(footprint "Connector_PinHeader_2.54mm:PinHeader_1x02_P2.54mm_Vertical"
 		(layer "F.Cu")
-		(at 170.434 100.198)
+		(at 170.307 100.198)
 		(descr "Through hole straight pin header, 1x02, 2.54mm pitch, single row")
 		(tags "Through hole pin header THT 1x02 2.54mm single row")
@@
 	(footprint "Connector_PinHeader_2.54mm:PinHeader_1x06_P2.54mm_Vertical"
 		(layer "F.Cu")
-		(at 133.096 91.821)
+		(at 133.223 91.821)
 		(descr "Through hole straight pin header, 1x06, 2.54mm pitch, single row")
 		(tags "Through hole pin header THT 1x06 2.54mm single row")
@@
 	(footprint "Library:AE-XC9306-5V0"
 		(layer "F.Cu")
-		(at 145.796 102.616 -90)
+		(at 145.796 102.362 -90)
 		(descr "6-lead though-hole mounted DIP package, row spacing 7.62 mm (300 mils), SMDSocket, SmallPads")
 		(tags "THT DIP DIL PDIP 2.54mm 7.62mm 300mil SMDSocket SmallPads")
 		(property "Reference" "IC2"
-			(at -0.381 2.667 180)
+			(at 0.254 0 180)
 			(layer "F.SilkS")
 			(effects
@@
 	)
 	(gr_text "S"
-		(at 142.0876 94.996 0)
+		(at 135.509 94.996 0)
 		(layer "B.SilkS")
 		(effects
@@
 	)
 	(gr_text "WS2812B"
-		(at 147.955 92.329 0)
+		(at 137.541 90.297 0)
 		(layer "B.SilkS")
 		(effects
 			(font
-				(size 1 1)
-				(thickness 0.15)
+				(size 0.6 0.6)
+				(thickness 0.075)
 			)
 			(justify left bottom mirror)
@@
 	)
 	(gr_text "RXD"
-		(at 143.891 100.076 0)
+		(at 135.990071 99.821 0)
 		(layer "B.SilkS")
 		(effects
 			(font
-				(size 1 1)
-				(thickness 0.15)
+				(size 0.6 0.6)
+				(thickness 0.075)
 			)
 			(justify left bottom mirror)
@@
 	)
 	(gr_text "TXD"
-		(at 143.764 97.536 0)
+		(at 135.990071 97.281 0)
 		(layer "B.SilkS")
 		(effects
 			(font
-				(size 1 1)
-				(thickness 0.15)
+				(size 0.6 0.6)
+				(thickness 0.075)
 			)
 			(justify left bottom mirror)
@@
 	)
 	(via
+		(at 135.509 89.027)
+		(size 0.8)
+		(drill 0.4)
+		(layers "F.Cu" "B.Cu")
+		(free yes)
+		(net 1)
+	)
+	(via
 		(at 155.829 91.948)
 		(size 0.8)
@@
 	)
 	(via
+		(at 145.161 100.965)
+		(size 0.8)
+		(drill 0.4)
+		(layers "F.Cu" "B.Cu")
+		(free yes)
+		(net 1)
+	)
+	(via
 		(at 149.479 91.948)
 		(size 0.8)
@@
 	)
 	(via
+		(at 164.592 101.473)
+		(size 0.8)
+		(drill 0.4)
+		(layers "F.Cu" "B.Cu")
+		(free yes)
+		(net 1)
+	)
+	(via
 		(at 166.497 89.662)
 		(size 0.8)
@@
 	)
 	(via
-		(at 166.497 105.918)
+		(at 166.497 106.299)
 		(size 0.8)
 		(drill 0.4)
@@
 	)
 	(segment
-		(start 166.751 96.647)
-		(end 164.719 98.679)
+		(start 168.529 101.981)
+		(end 168.529 98.425)
 		(width 0.25)
 		(layer "B.Cu")
@@
 	)
 	(segment
-		(start 164.719 101.854)
-		(end 165.608 102.743)
+		(start 168.529 98.425)
+		(end 166.751 96.647)
 		(width 0.25)
 		(layer "B.Cu")
@@
 	)
 	(segment
-		(start 164.719 98.679)
-		(end 164.719 101.854)
+		(start 167.767 102.743)
+		(end 168.529 101.981)
 		(width 0.25)
 		(layer "B.Cu")
@@
 	)
 	(segment
-		(start 165.608 102.743)
-		(end 166.751 102.743)
+		(start 166.751 102.743)
+		(end 167.767 102.743)
 		(width 0.25)
 		(layer "B.Cu")
