File: Pmod_Joystick/Pmod_Joystick.kicad_sch (KiCad schematic)
At the start: 12 parts, among them J1 JoyStick, J2 Conn_02x06_Top_Bottom, U1 MCP3004

Commit message: 1202
Connections:
- net Vcc: now reaches C1.1, C3.1, J2.12 (Pin_12), J2.6 (Pin_6), R1.1, U1.14 (Vdd)
Changed lines of the file:
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@@
+		)
+	)
+	(label "Vcc"
+		(at 102.87 99.695 0)
+		(fields_autoplaced yes)
+		(effects
+			(font
+				(size 1.27 1.27)
+			)
+			(justify left bottom)
 		)
 	)
