File: Pmod_SC1602/Pmod_SC1602.kicad_sch (KiCad schematic)
At the start: 12 parts, among them Q2 Q_NPN_BEC

Commit message: 0106
Parts:
- added J1: Pmod_Header, MyLibrary:Pmod, symbol MyLibrary:Pmod_Header
Changed lines of the file:
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@@
+    )
+  )
+  (symbol (lib_id "MyLibrary:Pmod_Header") (at 36.83 93.98 0) (unit 1)
+    (in_bom yes) (on_board yes) (dnp no) (fields_autoplaced)
+    (property "Reference" "J1" (at 38.1 80.01 0)
+      (effects (font (size 1.27 1.27)))
+    )
+    (property "Value" "Pmod_Header" (at 38.1 82.55 0)
+      (effects (font (size 1.27 1.27)))
+    )
+    (property "Footprint" "MyLibrary:Pmod" (at 38.1 85.09 0)
+      (effects (font (size 1.27 1.27)))
+    )
+    (property "Datasheet" "~" (at 36.83 93.98 0)
+      (effects (font (size 1.27 1.27)) hide)
+    )
+    (pin "9")
+    (pin "5")
+    (pin "7")
+    (pin "11")
+    (pin "8")
+    (pin "1")
+    (pin "6")
+    (pin "2")
+    (pin "4")
+    (pin "12")
+    (pin "3")
+    (pin "10")
+    (instances
+      (project "Pmod_SC1602"
+        (path "/f47043ba-0e76-4450-91ea-b39e58f9a09a"
+          (reference "J1") (unit 1)
+        )
+      )
     )
   )

Commit message: 0106
Connections:
- net BackLight: now also J1.10 (Pin_10)
- net Contrast: now also J1.9 (Pin_9)
- net D0: now also J1.1 (Pin_1)
- net D1: now also J1.7 (Pin_7)
- net D2: now also J1.2 (Pin_2)
- net D3: now also J1.8 (Pin_8)
- net GND: now also J1.11 (Pin_11), J1.5 (Pin_5)
- net RS: now also J1.3 (Pin_3)
- net R/W: now also J1.4 (Pin_4)
- net VCC: now also J1.12 (Pin_12), J1.6 (Pin_6)

Commit message: 1204
Parts:
- removed JP1: SolderJumper_2_Open, Jumper:SolderJumper-2_P1.3mm_Open_TrianglePad1.0x1.5mm, symbol Jumper:SolderJumper_2_Open
- removed JP3, JP4, JP5: SolderJumper_2_Bridged, Jumper:SolderJumper-2_P1.3mm_Bridged_RoundedPad1.0x1.5mm, symbol Jumper:SolderJumper_2_Bridged
- removed RV1: 20k, Potentiometer_THT:Potentiometer_Bourns_3266Z_Horizontal, symbol Device:R_Potentiometer_Small
- added C3: 1u, Capacitor_SMD:C_0603_1608Metric_Pad1.08x0.95mm_HandSolder, symbol Device:C
- added J2: Conn_01x02, Connector_PinSocket_2.54mm:PinSocket_1x02_P2.54mm_Vertical, symbol Connector_Generic:Conn_01x02
- added J3: Conn_01x03, Connector_PinSocket_2.54mm:PinSocket_1x03_P2.54mm_Vertical, symbol Connector_Generic:Conn_01x03
- added Q1: Q_NPN_BEC, Package_TO_SOT_SMD:SC-59_Handsoldering, symbol Device:Q_NPN_BEC
- added RV2: R_Potentiometer_Small, Potentiometer_THT:Potentiometer_Vishay_T73XW_Horizontal, symbol Device:R_Potentiometer_Small
- C1: value 1u -> 10u; footprint Capacitor_SMD:C_0603_1608Metric_Pad1.08x0.95mm_HandSolder -> Capacitor_SMD:C_0805_2012Metric_Pad1.18x1.45mm_HandSolder
Connections:
- net BackLight: now also R2.1; no longer JP2.2 (B)
- net Contrast: now also Q1.3 (C); no longer J1.9 (Pin_9)
- net D1: now also DS1.12 (DB5), J1.8 (Pin_8); no longer DS1.14 (DB7), J1.7 (Pin_7)
- net D3: now also DS1.14 (DB7), J1.7 (Pin_7); no longer DS1.12 (DB5), J1.8 (Pin_8)
- net GND: now also JP2.2 (B), C3.2, J3.3 (Pin_3), Q1.2 (E), RV2.3
- net R/W: now also J3.2 (Pin_2); no longer J1.4 (Pin_4)
- net VCC: now also C3.1
- net at C1.1, R1.2: now also J2.1 (Pin_1)
- net at DS1.3 (VO): now also J2.2 (Pin_2), RV2.2
- net at JP2.1 (A): now also DS1.K1, DS1.K2, Q2.3 (C); no longer DS1.6 (E)
- new net: J1.9 (Pin_9), J3.1 (Pin_1), Q1.1 (B)
- new net: DS1.6 (E), J1.4 (Pin_4)
- no-connect marks 4 -> 5
