File: Pmod_SC1602/Pmod_SC1602.kicad_pcb (KiCad board)
At the start: 2 copper layers, 99.9 x 32.6 mm, 12 parts, among them Q2 Q_NPN_BEC

Commit message: 0106
Parts:
- added J1: Pmod_Header, MyLibrary:Pmod, F.Cu at (83.4, 84.5)

Commit message: 0106
Parts:
- added JP6: SolderJumper_2_Open, Jumper:SolderJumper-2_P1.3mm_Open_TrianglePad1.0x1.5mm, F.Cu at (177.7, 89.0)
- added REF**: PinHeader_1x01_P2.54mm_Vertical, Connector_PinHeader_2.54mm:PinHeader_1x01_P2.54mm_Vertical, F.Cu at (152.0, 99.7)
- moved RV1 12.9 mm to (145.7, 97.2)
- moved J1 5.91 mm to (82.6, 90.3)
Connections:
- J1 pad 1: unconnected-(J1-Pin_1-Pad1) -> /D0
- J1 pad 10: unconnected-(J1-Pin_10-Pad10) -> /BackLight
- J1 pad 11: unconnected-(J1-Pin_11-Pad11) -> GND
- J1 pad 12: unconnected-(J1-Pin_12-Pad12) -> VCC
- J1 pad 2: unconnected-(J1-Pin_2-Pad2) -> /D2
- J1 pad 3: unconnected-(J1-Pin_3-Pad3) -> /RS
- J1 pad 4: unconnected-(J1-Pin_4-Pad4) -> /R/W
- J1 pad 5: unconnected-(J1-Pin_5-Pad5) -> GND
- J1 pad 6: unconnected-(J1-Pin_6-Pad6) -> VCC
- J1 pad 7: unconnected-(J1-Pin_7-Pad7) -> /D1
- J1 pad 8: unconnected-(J1-Pin_8-Pad8) -> /D3
- J1 pad 9: unconnected-(J1-Pin_9-Pad9) -> /Contrast
Routing:
- net VCC: track 59.6 -> 109.8 mm
- net /BackLight: track 4.60 -> 46.8 mm
- net /Contrast: track 0.00 -> 25.5 mm
- net Net-(JP1-B): track 19.7 -> 39.0 mm
- net /D2: track 0.00 -> 19.1 mm
- net /D3: track 0.00 -> 18.8 mm
- net /D1: track 0.00 -> 15.9 mm
- net /R/W: track 0.00 -> 13.6 mm
- net /D0: track 0.00 -> 13.6 mm
- net /RS: track 0.00 -> 9.11 mm
- net Net-(Q2-C): track 8.02 -> 15.2 mm
Other:
- board text added: "Anode"
- board text added: "BL"
- board text added: "BackLight(Pmod)<->BackLight(SC1602)"
- board text added: "BackLight(Pmod)<->E(SC1602)"
- board text added: "Cathode"
- board text added: "Co"
- board text added: "D0"
- board text added: "D1"
- board text added: "D2"
- board text added: "D3"
- board text added: "E(SC1602)<->GND"
- board text added: "GND"
- board text added: "GND<->Cathode(SC1602)"
- board text added: "Pmod_SC1602"
- board text added: "R/W"
- board text added: "RS"
- board text added: "VO"
- board text added: "VO(SC1602)<->Contrast(Pmod)"
- board text added: "VO(SC1602)<->RV1"
- board text added: "Vcc"
- board text removed: "Sugamod_SC1602"

Commit message: 0107
Parts:
- added G***: LOGO, MyLibrary:logo_kamo_ss, F.Cu at (93.3, 81.2)
- added G***: LOGO, MyLibrary:kamo20, B.Cu at (137.3, 89.8)
Routing:
- net /BackLight: track 46.8 -> 45.0 mm
- net GND: vias 0 -> 11

Commit message: 1204
Parts:
- removed JP1, JP6: SolderJumper_2_Open, Jumper:SolderJumper-2_P1.3mm_Open_TrianglePad1.0x1.5mm
- removed JP3, JP4, JP5: SolderJumper_2_Bridged, Jumper:SolderJumper-2_P1.3mm_Bridged_RoundedPad1.0x1.5mm
- removed REF**: PinHeader_1x01_P2.54mm_Vertical, Connector_PinHeader_2.54mm:PinHeader_1x01_P2.54mm_Vertical
- removed RV1: 20k, Potentiometer_THT:Potentiometer_Bourns_3266Z_Horizontal
- added C3: 1u, Capacitor_SMD:C_0603_1608Metric_Pad1.08x0.95mm_HandSolder, F.Cu at (108.5, 100.8)
- added J2: Conn_01x02, Connector_PinSocket_2.54mm:PinSocket_1x02_P2.54mm_Vertical, F.Cu at (120.8, 96.4)
- added J3: Conn_01x03, Connector_PinSocket_2.54mm:PinSocket_1x03_P2.54mm_Vertical, F.Cu at (114.6, 92.8)
- added Q1: Q_NPN_BEC, Package_TO_SOT_SMD:SC-59_Handsoldering, F.Cu at (127.4, 102.1)
- added RV2: R_Potentiometer_Small, Potentiometer_THT:Potentiometer_Vishay_T73XW_Horizontal, F.Cu at (114.7, 98.3)
- C1: value 1u -> 10u; footprint Capacitor_SMD:C_0603_1608Metric_Pad1.08x0.95mm_HandSolder -> Capacitor_SMD:C_0805_2012Metric_Pad1.18x1.45mm_HandSolder
- moved JP2 62.9 mm to (177.5, 88.9)
- moved R1 12.3 mm to (125.7, 97.3), turned to 90 degrees
- moved C1 10.2 mm to (128.5, 97.4), turned to -90 degrees
- moved G*** 5.72 mm to (143.0, 89.8)
- moved G*** 1.82 mm to (94.1, 82.8)
Connections:
- DS1 pad 12: /D3 -> /D1
- DS1 pad 14: /D1 -> /D3
- DS1 pad K1: Net-(Q2-C) -> Net-(JP2-A)
- DS1 pad K2: Net-(Q2-C) -> Net-(JP2-A)
- J1 pad 4: /R/W -> Net-(DS1-E)
- J1 pad 7: /D1 -> /D3
- J1 pad 8: /D3 -> /D1
- J1 pad 9: /Contrast -> Net-(J1-Pin_9)
- JP2 pad 1: Net-(DS1-E) -> Net-(JP2-A)
- JP2 pad 2: /BackLight -> GND
- Q2 pad 3: Net-(Q2-C) -> Net-(JP2-A)
- R2 pad 1: Net-(JP4-B) -> /BackLight
Routing:
- net Net-(J1-Pin_9): track 0.00 -> 76.6 mm
- net Net-(JP4-B): track 58.9 -> 0.00 mm
- net /BackLight: track 45.0 -> 100.0 mm
- net Net-(JP1-B): track 39.0 -> 0.00 mm
- net /Contrast: track 25.5 -> 3.91 mm
- net Net-(Q2-C): track 15.2 -> 0.00 mm
- net Net-(JP2-A): track 0.00 -> 15.2 mm
- net VCC: track 109.8 -> 117.3 mm
- net Net-(DS1-E): track 18.4 -> 11.1 mm
- net Net-(DS1-VO): track 13.9 -> 19.5 mm
- net /R/W: track 13.6 -> 10.2 mm
- net /D3: track 18.8 -> 15.9 mm
- net /D1: track 15.9 -> 18.3 mm
Other:
- board text added: "E"
- board text added: "GND<->SC1602_Cathode"
- board text added: "J2 - Pmod_Co <-> SC1602_VO"
- board text added: "Pmod_R/W"
- board text added: "Pmod_SC1602 Ver 0.2"
- board text added: "SC1602_R/W"
- board text removed: "BackLight(Pmod)<->BackLight(SC1602)"
- board text removed: "BackLight(Pmod)<->E(SC1602)"
- board text removed: "E(SC1602)<->GND"
- board text removed: "GND<->Cathode(SC1602)"
- board text removed: "Pmod_SC1602"
- board text removed: "VO(SC1602)<->Contrast(Pmod)"
- board text removed: "VO(SC1602)<->RV1"

Commit message: 1211
Routing:
- net Net-(J1-Pin_9): track 76.6 -> 77.5 mm
Other:
- board text added: "D4"
- board text added: "D5"
- board text added: "D6"
- board text added: "D7"
- board text removed: "D0"
- board text removed: "D2"
