File: Audio_Line/Audio_Line.kicad_pcb (KiCad board)
At the start: 2 copper layers, 43 parts, among them IC1 MCP6022-I_P, IC2 NJU7043D, J1 MJ-8435, J2 MJ-8435, J3 Conn_01x06, J4 Conn_01x06

Commit message: 0724
Parts:
- moved JP4 72.4 mm to (220.0, 112.0)
- moved JP14 62.0 mm to (223.5, 112.0)
- moved JP2 56.4 mm to (191.0, 109.0)
- moved R6 52.7 mm to (141.2, 63.5)
- moved R9 52.0 mm to (136.4, 70.4), turned to 180 degrees
- moved R10 50.5 mm to (136.0, 85.9)
- moved IC1 50.4 mm to (151.8, 67.6)
- moved RV1 48.9 mm to (148.8, 127.0)
- moved JP12 48.6 mm to (194.6, 109.0)
- moved R5 48.1 mm to (144.3, 64.5), turned to 90 degrees
- moved J2 47.9 mm to (209.3, 94.0), turned to -90 degrees
- moved JP3 46.6 mm to (175.3, 109.0)
- moved JP13 44.1 mm to (178.8, 109.0)
- moved J1 42.6 mm to (184.0, 73.7), turned to -90 degrees
- moved J4 41.2 mm to (125.8, 99.1), turned to 180 degrees
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Connections:
- R10 pad 1: unconnected-(R10-Pad1) -> /A0_IN
