File: Audio_Line/Audio_Line.kicad_sch (KiCad schematic)
At the start: 43 parts, among them IC1 MCP6022-I_P, IC2 NJU7043D, J1 MJ-8435, J2 MJ-8435, J3 Conn_01x06, J4 Conn_01x06

Commit message: 0724
Connections:
- net A0_IN: now also R10.1
Changed lines of the file:
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@@
+	(wire
+		(pts
+			(xy 159.385 81.915) (xy 161.925 81.915)
+		)
+		(stroke
+			(width 0)
+			(type default)
+		)
+	)
 	(wire
 		(pts
@@
 		)
 	)
+	(label "A0_IN"
+		(at 159.385 81.915 180)
+		(effects
+			(font
+				(size 1.27 1.27)
+			)
+			(justify right bottom)
+		)
+	)
