File: Pmod_PLED2/Pmod_PLED.kicad_sch (KiCad schematic)
At the start: 9 parts, among them IC1 TBD62064APG, J1 Barrel_Jack_Switch, J2 Conn_01x06_Pin, J3 Conn_01x03_Pin, U1 AMS1117-3.3

Commit message: power led 2 schematics
Parts:
- removed C1, C2: 0.1u, Capacitor_SMD:C_0603_1608Metric_Pad1.08x0.95mm_HandSolder, symbol Device:C
- removed D3: SS2040FL, SamacSys_Parts:SODFL3618X108N, symbol SamacSys_Parts:SS2040FL
- removed IC1: TBD62064APG, SamacSys_Parts:DIP762W60P254L1975H445Q16N, symbol SamacSys_Parts:TBD62064APG
- removed J1: Barrel_Jack_Switch, Connector_BarrelJack:BarrelJack_Horizontal, symbol Connector:Barrel_Jack_Switch
- removed J3: Conn_01x03_Pin, Connector_PinHeader_2.54mm:PinHeader_1x03_P2.54mm_Vertical, symbol Connector:Conn_01x03_Pin
- removed U1: AMS1117-3.3, Package_TO_SOT_SMD:SOT-223-3_TabPin2, symbol Regulator_Linear:AMS1117-3.3
- added R1, R2, R3: 10, symbol Device:R
- added U1, U2, U3: NJW4617, Package_TO_SOT_SMD:TO-252-5_TabPin3, symbol MyLibrary:NJW4617DL3
Connections:
- net Anode is gone; now on net VCC: D1.6 (A)
- net GND: now also R1.1, R2.1, R3.1, U1.3 (GND), U2.3 (GND), U3.3 (GND)
- net VCC: now also D1.4 (RA), U1.1 (VDD), U2.1 (VDD), U3.1 (VDD)
- net Anode_G: now reaches D1.1 (GK)
- net Anode_G: now also U2.5 (LED)
- net Anode_R: now reaches D1.2 (RK)
- net Anode_R: now also D1.5 (RK), U1.5 (LED)
- net Anode_B: now reaches D1.3 (BK)
- net Anode_B: now also U3.5 (LED)
- new net: R3.2, U3.4 (Rs)
- new net: R1.2, U2.4 (Rs)
- new net: R2.2, U1.4 (Rs)
- no-connect marks 4 -> 0
Other:
- moved on the sheet: D1, J2

Commit message: schematcis
Parts:
- added Q1, Q2, Q3: 2SC2712-BL_F_, samacsys:RN1402LF, symbol samacsys:2SC2712-BL_F_
- added R4, R5, R6: 10k, Resistor_SMD:R_0603_1608Metric_Pad0.98x0.95mm_HandSolder, symbol Device:R
- R1, R2, R3: footprint (none) -> Resistor_SMD:R_0603_1608Metric_Pad0.98x0.95mm_HandSolder
Connections:
- net GND: now also Q1.2 (E), Q2.2 (E), Q3.2 (E)
- net VCC: now also R4.1, R5.1, R6.1
- net EN_R: now reaches J2.1 (Pin_1)
- net EN_R: now also Q1.1 (B)
- net EN_G: now reaches J2.2 (Pin_2)
- net EN_G: now also Q2.1 (B)
- net EN_B: now reaches J2.3 (Pin_3)
- net EN_B: now also Q3.1 (B)
- net at U3.2 (EN/PWM): now also Q3.3 (C), R6.2
- net at U1.2 (EN/PWM): now also Q1.3 (C), R4.2
- net at U2.2 (EN/PWM): now also Q2.3 (C), R5.2
- no-connect marks 0 -> 1
Other:
- moved on the sheet: R1, R2, R3, U1, U2, U3
