File: Pmod_PLED2/Pmod_PLED.kicad_sch (KiCad schematic)
At the start: 23 parts, among them J2 Conn_01x06_Pin, Q1 2SC2712-BL_F_, Q2 2SC2712-BL_F_, Q3 2SC2712-BL_F_, U1 NJW4617, U2 NJW4617, U3 NJW4617

Commit message: 1109
Parts:
- removed Q1, Q2, Q3: 2SC2712-BL_F_, samacsys:RN1402LF, symbol samacsys:2SC2712-BL_F_
- removed R12, R13, R9: 4.7k, Resistor_SMD:R_0603_1608Metric_Pad0.98x0.95mm_HandSolder, symbol Device:R
- added Q1, Q2, Q4: BSS84, Package_TO_SOT_SMD:TSOT-23_HandSoldering, symbol Transistor_FET:BSS84
- D1: footprint MyLibrary:EP204-150G1R1B1-CA -> kicad8-2:EP204-150G1R1B1-CA
- J2: footprint Library:Pmod6 -> Connector_PinHeader_2.54mm:PinHeader_1x06_P2.54mm_Vertical_SMD_Pin1Left
Connections:
- net EN_B: now also Q2.2 (S)
- net EN_G: now also Q1.2 (S)
- net EN_R: now also Q4.2 (S)
- net at R6.2, U3.2 (EN/PWM): now also Q2.3 (D)
- net at R14.1, R15.2: now also Q2.1 (G)
- net at R5.2, U2.2 (EN/PWM): now also Q1.3 (D)
- net at R7.1, R8.2: now also Q4.1 (G)
- net at R4.2, U1.2 (EN/PWM): now also Q4.3 (D)
- net at R10.1, R11.2: now also Q1.1 (G)

Commit message: 1110
Connections:
- net VCC is gone; now on net EN_B: J2.6 (Pin_6)
- net 5V: now also J2.1 (Pin_1); no longer D1.1 (GK), U2.5 (LED)
- net EN_B: no longer J2.3 (Pin_3)
- net EN_G: now also J2.4 (Pin_4); no longer J2.2 (Pin_2)
- net EN_R: now also J2.2 (Pin_2); no longer J2.1 (Pin_1)
- net Anode_B renamed Cathode_B
- net Cathode_B: now also D1.1 (GK); no longer D1.3 (BK)
- net Anode_R renamed Cathode_R
- new net Cathode_G: D1.3 (BK), U2.5 (LED)
- no-connect marks 1 -> 0
