File: Pmod_PLED2/Pmod_PLED.kicad_pcb (KiCad board)
At the start: 2 copper layers, 74.5 x 20.3 mm, 10 parts, among them IC1 TBD62064APG, J1 Barrel_Jack_Switch, J2 Conn_01x06_Pin, J3 Conn_01x03_Pin, U1 AMS1117-3.3

Commit message: power led 2 schematics
Parts:
- removed D1: EP204K-150G1R1B1-CA, MyLibrary:EP204-150G1R1B1-CA
- removed D3: SS2040FL, SamacSys_Parts:SODFL3618X108N
- removed G***: LOGO, MyLibrary:logo_kamo_ss
- removed IC1: TBD62064APG, SamacSys_Parts:DIP762W60P254L1975H445Q16N
- removed J1: Barrel_Jack_Switch, Connector_BarrelJack:BarrelJack_Horizontal
- removed J2: Conn_01x06_Pin, Library:Pmod6
- removed J3: Conn_01x03_Pin, Connector_PinHeader_2.54mm:PinHeader_1x03_P2.54mm_Vertical
- U1: value AMS1117-3.3 -> NJW4617; footprint Package_TO_SOT_SMD:SOT-223-3_TabPin2 -> Package_TO_SOT_SMD:TO-252-5_TabPin3
- moved C1 43.0 mm to (117.2, 85.8), turned to 0 degrees
- moved U1 32.6 mm to (121.9, 80.5), turned to 0 degrees
- moved C2 32.3 mm to (117.2, 88.3), turned to 0 degrees
Connections:
- C1 pad 1: Net-(U1-VI) -> unconnected-(C1-Pad1)
- C2 pad 2: /ExVcc -> unconnected-(C2-Pad2)
- U1 pad 1: GND -> unconnected-(U1-VDD-Pad1)
- U1 pad 2: /ExVcc -> unconnected-(U1-EN/PWM-Pad2)
- U1 pad 3: Net-(U1-VI) -> unconnected-(U1-GND-Pad3)
Routing:
- net vcc: track 61.7 -> 0.00 mm
- net Net-(U1-VI): track 32.8 -> 0.00 mm
- net Net-(D1-BK): track 26.8 -> 0.00 mm
- net /Anode: track 21.2 -> 0.00 mm
- net i4: track 19.4 -> 0.00 mm
- net i1: track 17.8 -> 0.00 mm
- net /ExVcc: track 13.2 -> 0.00 mm
- net i3: track 11.0 -> 0.00 mm
- net i2: track 10.4 -> 0.00 mm
- net Net-(D1-GK): track 9.18 -> 0.00 mm
- net Net-(IC1-O4): track 6.20 -> 0.00 mm
- net Net-(D1-RA): track 3.37 -> 0.00 mm
- removed copper zone on F.Cu, net GND
Other:
- board outline removed
- board text removed: "1"
- board text removed: "2"
- board text removed: "3"
- board text removed: "4"
- board text removed: "ExVcc"
- board text removed: "GND"
- board text removed: "[AZ1117 CH-3.3]"
- board text removed: "[TBD62064APG]"
- board text removed: "i1"
- board text removed: "i2"
- board text removed: "i3"
- board text removed: "i4"
- board text removed: "in"
- board text removed: "o1"
- board text removed: "o2"
- board text removed: "o3"
- board text removed: "o4"
- board text removed: "out"

Commit message: schematcis
Parts:
- added Q1: 2SC2712-BL_F_, samacsys:RN1402LF, F.Cu at (140.7, 54.5)
- added Q2: 2SC2712-BL_F_, samacsys:RN1402LF, F.Cu at (146.7, 54.5)
- added Q3: 2SC2712-BL_F_, samacsys:RN1402LF, F.Cu at (152.7, 54.5)
- added R1: 10, Resistor_SMD:R_0603_1608Metric_Pad0.98x0.95mm_HandSolder, F.Cu at (152.0, 59.1)
- added R2: 10, Resistor_SMD:R_0603_1608Metric_Pad0.98x0.95mm_HandSolder, F.Cu at (152.0, 61.6)
- added R3: 10, Resistor_SMD:R_0603_1608Metric_Pad0.98x0.95mm_HandSolder, F.Cu at (152.0, 64.1)
- added R4: 10k, Resistor_SMD:R_0603_1608Metric_Pad0.98x0.95mm_HandSolder, F.Cu at (152.0, 66.6)
- added R5: 10k, Resistor_SMD:R_0603_1608Metric_Pad0.98x0.95mm_HandSolder, F.Cu at (152.0, 69.1)
- added R6: 10k, Resistor_SMD:R_0603_1608Metric_Pad0.98x0.95mm_HandSolder, F.Cu at (152.0, 71.6)
- added U2: NJW4617, Package_TO_SOT_SMD:TO-252-5_TabPin3, F.Cu at (144.6, 61.8)
- added U3: NJW4617, Package_TO_SOT_SMD:TO-252-5_TabPin3, F.Cu at (144.6, 69.9)
Connections:
- U1 pad 1: unconnected-(U1-VDD-Pad1) -> /VCC
- U1 pad 2: unconnected-(U1-EN/PWM-Pad2) -> Net-(Q1-C)
- U1 pad 3: unconnected-(U1-GND-Pad3) -> GND
- U1 pad 4: unconnected-(U1-Rs-Pad4) -> Net-(U1-Rs)
- U1 pad 5: unconnected-(U1-LED-Pad5) -> /Anode_R

Commit message: 1109
Parts:
- removed Q3: 2SC2712-BL_F_, samacsys:RN1402LF
- added D1: EP204K-150G1R1B1-CA, kicad8-2:EP204-150G1R1B1-CA, F.Cu at (114.4, 64.3)
- added J2: Conn_01x06_Pin, Connector_PinHeader_2.54mm:PinHeader_1x06_P2.54mm_Vertical_SMD_Pin1Left, F.Cu at (76.5, 63.4)
- added Q4: BSS84, Package_TO_SOT_SMD:TSOT-23_HandSoldering, F.Cu at (59.0, 88.4)
- added R10: 3.3k, Resistor_SMD:R_0603_1608Metric_Pad0.98x0.95mm_HandSolder, F.Cu at (82.7, 61.0)
- added R11: 2.2k, Resistor_SMD:R_0603_1608Metric_Pad0.98x0.95mm_HandSolder, F.Cu at (82.7, 63.6)
- added R14: 3.3k, Resistor_SMD:R_0603_1608Metric_Pad0.98x0.95mm_HandSolder, F.Cu at (82.7, 66.1)
- added R15: 2.2k, Resistor_SMD:R_0603_1608Metric_Pad0.98x0.95mm_HandSolder, F.Cu at (82.7, 68.6)
- added R7: 3.3k, Resistor_SMD:R_0603_1608Metric_Pad0.98x0.95mm_HandSolder, F.Cu at (82.7, 56.0)
- added R8: 2.2k, Resistor_SMD:R_0603_1608Metric_Pad0.98x0.95mm_HandSolder, F.Cu at (82.7, 58.5)
- Q1, Q2: value 2SC2712-BL_F_ -> BSS84; footprint samacsys:RN1402LF -> Package_TO_SOT_SMD:TSOT-23_HandSoldering
- moved Q2 92.4 mm to (59.0, 83.7)
- moved Q1 85.3 mm to (59.0, 79.1)
Connections:
- net /VCC renamed /5V
- Q1 pad 1: /EN_R -> Net-(Q1-G)
- Q1 pad 2: GND -> /EN_G
- Q1 pad 3: Net-(Q1-C) -> Net-(Q1-D)
- Q2 pad 1: /EN_G -> Net-(Q2-G)
- Q2 pad 2: GND -> /EN_B
- Q2 pad 3: Net-(Q2-C) -> Net-(Q2-D)
- R4 pad 2: Net-(Q1-C) -> Net-(Q4-D)
- R5 pad 2: Net-(Q2-C) -> Net-(Q1-D)
- R6 pad 2: Net-(Q3-C) -> Net-(Q2-D)
- U1 pad 2: Net-(Q1-C) -> Net-(Q4-D)
- U2 pad 2: Net-(Q2-C) -> Net-(Q1-D)
- U2 pad 5: /Anode_G -> Net-(D1-GK)
- U3 pad 2: Net-(Q3-C) -> Net-(Q2-D)

Commit message: 1110
Parts:
- removed C1, C2: 0.1u, Capacitor_SMD:C_0603_1608Metric_Pad1.08x0.95mm_HandSolder
- added REF**: MountingHole_4.3mm_M4, MountingHole:MountingHole_4.3mm_M4, F.Cu at (124.6, 104.7)
- added REF**: TestPoint_Pad_1.0x1.0mm, TestPoint:TestPoint_Pad_1.0x1.0mm, F.Cu at (137.3, 69.2)
- added REF**: TestPoint_Pad_2.0x2.0mm, TestPoint:TestPoint_Pad_2.0x2.0mm, F.Cu at (138.2, 105.4)
- added REF**: MountingHole_4.3mm_M4, MountingHole:MountingHole_4.3mm_M4, F.Cu at (159.6, 73.7)
- moved Q2 100.4 mm to (157.7, 102.3), turned to 180 degrees
- moved R15 85.8 mm to (159.5, 106.9), turned to 180 degrees
- moved R14 82.1 mm to (153.9, 106.8), turned to 180 degrees
- moved Q1 81.7 mm to (140.4, 72.2), turned to 180 degrees
- moved R11 64.4 mm to (146.0, 75.2), turned to 180 degrees
- moved J2 64.2 mm to (140.7, 66.0), turned to 90 degrees
- moved Q4 62.7 mm to (121.6, 90.4), turned to 90 degrees
- moved R10 59.8 mm to (140.8, 75.2), turned to 180 degrees
- moved R8 55.5 mm to (125.7, 93.5), turned to -90 degrees
- moved R7 53.8 mm to (119.4, 95.4), turned to 180 degrees
- moved R2 38.0 mm to (125.8, 89.1)
- moved R4 37.9 mm to (119.4, 86.0)
- moved D1 37.0 mm to (141.9, 89.2), turned to 180 degrees
- moved R3 34.2 mm to (153.0, 98.3), turned to 90 degrees
- moved R6 31.6 mm to (153.0, 103.2), turned to 90 degrees
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Connections:
- net /Anode_R renamed /Cathode_R
- D1 pad 1: Net-(D1-GK) -> /Cathode_B
- D1 pad 3: /Anode_B -> /Cathode_G
- J2 pad 1: /EN_R -> /5V
- J2 pad 2: /EN_G -> /EN_R
- J2 pad 3: /EN_B -> unconnected-(J2-Pin_3-Pad3)
- J2 pad 4: unconnected-(J2-Pin_4-Pad4) -> /EN_G
- J2 pad 6: /VCC -> /EN_B
- U2 pad 5: Net-(D1-GK) -> /Cathode_G
- U3 pad 5: /Anode_B -> /Cathode_B
Routing:
- net GND: track 0.00 -> 176.3 mm
- net /5V: track 0.00 -> 99.2 mm
- net /EN_B: track 0.00 -> 43.3 mm
- net /Cathode_G: track 0.00 -> 14.3 mm
- net Net-(Q4-G): track 0.00 -> 11.8 mm
- net Net-(Q2-D): track 0.00 -> 8.69 mm
- net Net-(Q4-D): track 0.00 -> 7.96 mm
- net /Cathode_R: track 0.00 -> 7.93 mm
- net Net-(Q2-G): track 0.00 -> 7.82 mm
- net /EN_G: track 0.00 -> 7.01 mm
- net Net-(U1-Rs): track 0.00 -> 5.91 mm
- net /Cathode_B: track 0.00 -> 5.53 mm
- net Net-(Q1-G): track 0.00 -> 5.44 mm
- net Net-(U3-Rs): track 0.00 -> 5.18 mm
- net Net-(Q1-D): track 0.00 -> 5.07 mm
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Other:
- board outline added: 53.7 x 58 mm
- board text added: "@1"
- board text added: "@2"
- board text added: "@3"
- board text added: "B"
- board text added: "Color_LED Ver. 0.1"
- board text added: "G"
- board text added: "GND"
- board text added: "R"
- board text removed: "Pmod_Color_LED Ver. 0.2"
- board text removed: "[EP204K- 150G1R1B1-CA]"
